File: td-io.sch (KiCad schematic (older format))
At the start: 58 parts, among them J1 USB_A, J2 USB_B, J3 JAMMA_Edge, J4 AudioJack3, J5 DB15_Male_HighDensity, J6 Conn_02x04_Top_Bottom, Q1 Si7141DP, U1 AD813, U2 AD813, U3 AD813, U4 74LS86, U5 AD813, U6 STM32L031C6Tx, U7 LM25085MM

Commit message: Update schematic
Parts:
- removed C10, C11, C9: 0.1uF, symbol Device:C
- removed U6: STM32L031C6Tx, Package_QFP:LQFP-48_7x7mm_P0.5mm, symbol MCU_ST_STM32L0:STM32L031C6Tx
- added D2: BAT54A, Package_TO_SOT_SMD:SOT-23, symbol Diode:BAT54A
- added J7: Conn_02x17_Odd_Even, td-io:DF1BZ-34DP-2.5DSA, symbol Connector_Generic:Conn_02x17_Odd_Even
- added Q2, Q3: FDS6930A, Package_SO:SOIC-8_3.9x4.9mm_P1.27mm, symbol Transistor_FET:FDS6930A
- added R25, R26: 1k, Resistor_SMD:R_0805_2012Metric, symbol Device:R
- added RV1: 10k Audio, Potentiometer_THT:Potentiometer_Alps_RK09K_Single_Vertical, symbol Device:R_POT
- added SW1: SW_DIP_x02, Button_Switch_SMD:SW_DIP_SPSTx02_Slide_Omron_A6S-210x_W8.9mm_P2.54mm, symbol Switch:SW_DIP_x02
- added U10: Pico, MCU_RaspberryPi_and_Boards:RPi_Pico_SMD_TH, symbol MCU_RaspberryPi_and_Boards:Pico
- added U6, U8, U9: 74LV166, Package_SO:SOIC-16_3.9x9.9mm_P1.27mm, symbol 74xx:74LS166
- C1, C12, C13, C14, C15, C17, C18, C2, C3, C4, C5, C6, C7: footprint (none) -> Capacitor_SMD:C_0805_2012Metric
- C16: footprint (none) -> Capacitor_SMD:CP_Elec_5x5.3; Digikey (none) -> 732-6394-2-ND
- C8: value 0.1uF -> 1uF; footprint (none) -> Capacitor_SMD:C_0805_2012Metric
- D1: footprint (none) -> Diode_SMD:D_SMC; Digikey (none) -> SL44-E3/57TGICT-ND
- J1: footprint (none) -> Connector_USB:USB_A_Molex_67643_Horizontal
- J2: footprint (none) -> Connector_USB:USB_B_OST_USB-B1HSxx_Horizontal
- J3: footprint (none) -> td-io:JAMMA
- J4: footprint (none) -> Connector_Audio:Jack_3.5mm_CUI_SJ-3523-SMT_Horizontal
- J5: footprint (none) -> Connector_Dsub:DSUB-15-HD_Male_Horizontal_P2.29x1.98mm_EdgePinOffset3.03mm_Housed_MountingHolesOffset4.94mm
- J6: footprint (none) -> td-io:B08P-VL
- L1: value 0.68mH -> 0.1mH; footprint (none) -> Inductor_THT:L_Toroid_Horizontal_D32.5mm_P30.00mm_Bourns_2300; Digikey (none) -> 2312-H-RC
- R1, R10, R11, R12, R13, R14, R15, R16, R17, R18, R19, R2, R20, R21, R22, R23, R24, R3, R4, R5, R6, R7, R8, R9: footprint (none) -> Resistor_SMD:R_0805_2012Metric
- U1: value AD813 -> LM4950TS; footprint (none) -> Package_TO_SOT_SMD:TO-263-9_TabPin5
- U2: value AD813 -> ST485EB; footprint (none) -> Package_SO:SOIC-8_3.9x4.9mm_P1.27mm
- U3, U4: footprint (none) -> Package_SO:SOIC-14_3.9x8.7mm_P1.27mm
- U5: footprint (none) -> Package_SO:SOIC-8_3.9x4.9mm_P1.27mm
Connections:
- net labels added: lockout1, lockout1_ctl, lockout2, lockout2_ctl, meter1, meter1_ctl, meter2, meter2_ctl, p1_5, p1_6, p2_5, p2_6, sr_clk, sr_clr, sr_data
- wire segments 243 -> 273
- no-connect marks 3 -> 36
Other:
- note removed: "addreset\nadd programming connector\nadd boot0 switch"
- note removed: "todo add mixer\ntodo add volume control"
- moved on the sheet: C2

Commit message: Swap male to female VGA connector
Parts:
- removed J5: DB15_Male_HighDensity, Connector_Dsub:DSUB-15-HD_Male_Horizontal_P2.29x1.98mm_EdgePinOffset3.03mm_Housed_MountingHolesOffset4.94mm, symbol Connector:DB15_Male_HighDensity
- added J5: DB15_Female_HighDensity, Connector_Dsub:DSUB-15-HD_Female_Horizontal_P2.29x1.98mm_EdgePinOffset3.03mm_Housed_MountingHolesOffset4.94mm, symbol Connector:DB15_Female_HighDensity
Connections:
- wire segments 273 -> 271
Other:
- note removed: "todo switch to female"
Changed lines of the file:
@@
 Connection ~ 15050 1400
-$Comp
-L Connector:DB15_Male_HighDensity J5
-U 1 1 6009D527
-P 4900 6550
-F 0 "J5" H 4900 7417 50  0000 C CNN
-F 1 "DB15_Male_HighDensity" H 4900 7326 50  0000 C CNN
-F 2 "Connector_Dsub:DSUB-15-HD_Male_Horizontal_P2.29x1.98mm_EdgePinOffset3.03mm_Housed_MountingHolesOffset4.94mm" H 3950 6950 50  0001 C CNN
-F 3 " ~" H 3950 6950 50  0001 C CNN
-	1    4900 6550
-	1    0    0    -1
-$EndComp
-$Comp
-L Memory_EEPROM:AT24CS01-SSHM U5
-U 1 1 600A0D28
-P 6100 6450
-F 0 "U5" H 6200 6900 50  0000 C CNN
-F 1 "AD813" H 6500 6750 50  0000 C CNN
-F 2 "Package_SO:SOIC-8_3.9x4.9mm_P1.27mm" H 6100 6450 50  0001 C CNN
-F 3 "http://ww1.microchip.com/downloads/en/DeviceDoc/Atmel-8815-SEEPROM-AT24CS01-02-Datasheet.pdf" H 6100 6450 50  0001 C CNN
-	1    6100 6450
-	1    0    0    -1
-$EndComp
-Text Label 4600 6850 2    50   ~ 0
-vga_red
-Text Label 4600 6650 2    50   ~ 0
-vga_green
-Text Label 4600 6450 2    50   ~ 0
-vga_blue
-Text Label 5200 6450 0    50   ~ 0
-vga_hsync
-Text Notes 4500 7300 0    50   ~ 0
-todo switch to female
-$Comp
-L power:GND #PWR0124
-U 1 1 600A33F9
-P 6100 6900
-F 0 "#PWR0124" H 6100 6650 50  0001 C CNN
-F 1 "GND" H 6105 6727 50  0000 C CNN
-F 2 "" H 6100 6900 50  0001 C CNN
-F 3 "" H 6100 6900 50  0001 C CNN
-	1    6100 6900
-	1    0    0    -1
-$EndComp
-Wire Wire Line
-	6100 6750 6100 6850
-Wire Wire Line
-	6100 6750 5650 6750
-Wire Wire Line
-	5650 6750 5650 6550
-Wire Wire Line
-	5650 6550 5700 6550
-Connection ~ 6100 6750
-Wire Wire Line
-	5650 6550 5650 6450
-Wire Wire Line
-	5650 6450 5700 6450
-Connection ~ 5650 6550
-Wire Wire Line
-	5650 6450 5650 6350
-Wire Wire Line
-	5650 6350 5700 6350
-Connection ~ 5650 6450
-$Comp
-L power:GND #PWR0125
-U 1 1 600AC403
-P 4150 6150
-F 0 "#PWR0125" H 4150 5900 50  0001 C CNN
-F 1 "GND" H 4155 5977 50  0000 C CNN
-F 2 "" H 4150 6150 50  0001 C CNN
-F 3 "" H 4150 6150 50  0001 C CNN
-	1    4150 6150
-	1    0    0    -1
-$EndComp
-Wire Wire Line
-	4150 6150 4250 6150
-Wire Wire Line
-	4250 6150 4250 6550
-Wire Wire Line
-	4250 6750 4600 6750
-Connection ~ 4250 6150
-Wire Wire Line
-	4250 6150 4600 6150
-Wire Wire Line
-	4600 6950 4250 6950
-Wire Wire Line
-	4250 6950 4250 6750
-Connection ~ 4250 6750
-Wire Wire Line
-	4600 6550 4250 6550
-Connection ~ 4250 6550
-Wire Wire Line
-	4250 6550 4250 6750
-Wire Wire Line
-	4600 6050 4250 6050
-Wire Wire Line
-	4250 6050 4250 6150
-Wire Wire Line
-	4600 6350 4350 6350
-Wire Wire Line
-	4350 6350 4350 5500
-Wire Wire Line
-	4350 5500 6100 5500
-Wire Wire Line
-	6100 5500 6100 6150
-Wire Wire Line
-	5200 6050 6600 6050
-Wire Wire Line
-	6600 6050 6600 6450
-Wire Wire Line
-	6600 6450 6500 6450
-Wire Wire Line
-	5200 6650 5550 6650
-Wire Wire Line
-	5550 6650 5550 7250
-Wire Wire Line
-	5550 7250 6650 7250
-Wire Wire Line
-	6650 7250 6650 6350
-Wire Wire Line
-	6650 6350 6500 6350
-Wire Wire Line
-	6100 6750 6500 6750
-Wire Wire Line
-	6500 6750 6500 6550
-NoConn ~ 4600 6250
-NoConn ~ 5200 6250
 $Comp
 L Amplifier_Video:AD813 U3
@@
 	1    0    0    -1
 $EndComp
-$Comp
-L Device:C C7
-U 1 1 60034C1D
-P 6850 6450
-F 0 "C7" H 6965 6496 50  0000 L CNN
-F 1 "0.1uF" H 6965 6405 50  0000 L CNN
-F 2 "Capacitor_SMD:C_0805_2012Metric" H 6888 6300 50  0001 C CNN
-F 3 "~" H 6850 6450 50  0001 C CNN
-	1    6850 6450
-	1    0    0    -1
-$EndComp
-Wire Wire Line
-	6850 6300 6850 5500
-Wire Wire Line
-	6850 5500 6100 5500
-Connection ~ 6100 5500
-Wire Wire Line
-	6100 6850 6850 6850
-Wire Wire Line
-	6850 6850 6850 6600
-Connection ~ 6100 6850
-Wire Wire Line
-	6100 6850 6100 6900
 $Comp
 L Device:C C6
@@
 Text Label 5550 10350 2    50   ~ 0
 vga_vsync
-Text Label 5200 6850 0    50   ~ 0
-vga_vsync
 $Comp
 L Device:R R6
@@
 	14250 2800 14250 2500
 Connection ~ 14250 2500
-$Comp
-L power:PWR_FLAG #FLG0101
-U 1 1 602B1EF0
-P 6100 5500
-F 0 "#FLG0101" H 6100 5575 50  0001 C CNN
-F 1 "PWR_FLAG" H 6100 5673 50  0000 C CNN
-F 2 "" H 6100 5500 50  0001 C CNN
-F 3 "~" H 6100 5500 50  0001 C CNN
-	1    6100 5500
-	1    0    0    -1
-$EndComp
 $Comp
 L MCU_RaspberryPi_and_Boards:Pico U10
@@
 	9950 6900 9950 6800
 Connection ~ 9950 6900
+$Comp
+L Connector:DB15_Female_HighDensity J5
+U 1 1 607A4CC7
+P 5050 6700
+F 0 "J5" H 5050 7567 50  0000 C CNN
+F 1 "DB15_Female_HighDensity" H 5050 7476 50  0000 C CNN
+F 2 "Connector_Dsub:DSUB-15-HD_Female_Horizontal_P2.29x1.98mm_EdgePinOffset3.03mm_Housed_MountingHolesOffset4.94mm" H 4100 7100 50  0001 C CNN
+F 3 " ~" H 4100 7100 50  0001 C CNN
+	1    5050 6700
+	1    0    0    -1
+$EndComp
+$Comp
+L Memory_EEPROM:AT24CS01-SSHM U5
+U 1 1 607C39AA
+P 6200 6700
+F 0 "U5" H 6300 7150 50  0000 C CNN
+F 1 "AD813" H 6600 7000 50  0000 C CNN
+F 2 "Package_SO:SOIC-8_3.9x4.9mm_P1.27mm" H 6200 6700 50  0001 C CNN
+F 3 "http://ww1.microchip.com/downloads/en/DeviceDoc/Atmel-8815-SEEPROM-AT24CS01-02-Datasheet.pdf" H 6200 6700 50  0001 C CNN
+	1    6200 6700
+	1    0    0    -1
+$EndComp
+Wire Wire Line
+	5350 7100 6800 7100
+Wire Wire Line
+	6800 7100 6800 6700
+Wire Wire Line
+	6800 6700 6600 6700
+$Comp
+L power:GND #PWR02
+U 1 1 607D8BDF
+P 6200 7200
+F 0 "#PWR02" H 6200 6950 50  0001 C CNN
+F 1 "GND" H 6205 7027 50  0000 C CNN
+F 2 "" H 6200 7200 50  0001 C CNN
+F 3 "" H 6200 7200 50  0001 C CNN
+	1    6200 7200
+	1    0    0    -1
+$EndComp
+Wire Wire Line
+	6200 7200 6200 7150
+Wire Wire Line
+	6600 6800 6600 7000
+Wire Wire Line
+	6600 7000 6200 7000
+Connection ~ 6200 7000
+Wire Wire Line
+	6200 7000 5800 7000
+Wire Wire Line
+	5800 7000 5800 6800
+Wire Wire Line
+	5800 6800 5800 6700
+Connection ~ 5800 6800
+Wire Wire Line
+	5800 6700 5800 6600
+Connection ~ 5800 6700
+Wire Wire Line
+	6600 6600 6800 6600
+Wire Wire Line
+	6800 6600 6800 6350
+Wire Wire Line
+	6800 6350 5600 6350
+Wire Wire Line
+	5600 6350 5600 6500
+Wire Wire Line
+	5600 6500 5350 6500
+$Comp
+L power:PWR_FLAG #FLG01
+U 1 1 60855E9C
+P 6200 5850
+F 0 "#FLG01" H 6200 5925 50  0001 C CNN
+F 1 "PWR_FLAG" H 6200 6023 50  0000 C CNN
+F 2 "" H 6200 5850 50  0001 C CNN
+F 3 "~" H 6200 5850 50  0001 C CNN
+	1    6200 5850
+	1    0    0    -1
+$EndComp
+Wire Wire Line
+	6200 6400 6200 6000
+Wire Wire Line
+	4750 6800 4350 6800
+Wire Wire Line
+	4350 6800 4350 6000
+Wire Wire Line
+	4350 6000 6200 6000
+Connection ~ 6200 6000
+Wire Wire Line
+	6200 6000 6200 5850
+Text Label 5350 6700 0    50   ~ 0
+vga_hsync
+Text Label 5350 6300 0    50   ~ 0
+vga_vsync
+Text Label 4750 6700 2    50   ~ 0
+vga_blue
+Text Label 4750 6500 2    50   ~ 0
+vga_green
+Text Label 4750 6300 2    50   ~ 0
+vga_red
+$Comp
+L power:GND #PWR01
+U 1 1 608837A8
+P 4250 7250
+F 0 "#PWR01" H 4250 7000 50  0001 C CNN
+F 1 "GND" H 4255 7077 50  0000 C CNN
+F 2 "" H 4250 7250 50  0001 C CNN
+F 3 "" H 4250 7250 50  0001 C CNN
+	1    4250 7250
+	1    0    0    -1
+$EndComp
+Wire Wire Line
+	4750 7100 4250 7100
+Wire Wire Line
+	4250 7100 4250 7250
+Wire Wire Line
+	4750 6200 4250 6200
+Wire Wire Line
+	4250 6200 4250 6400
+Connection ~ 4250 7100
+Wire Wire Line
+	4750 7000 4250 7000
+Connection ~ 4250 7000
+Wire Wire Line
+	4250 7000 4250 7100
+Wire Wire Line
+	4750 6600 4250 6600
+Connection ~ 4250 6600
+Wire Wire Line
+	4250 6600 4250 7000
+Wire Wire Line
+	4750 6400 4250 6400
+Connection ~ 4250 6400
+Wire Wire Line
+	4250 6400 4250 6600
+NoConn ~ 4750 6900
+NoConn ~ 5350 6900
+$Comp
+L Device:C C7
+U 1 1 6092E164
+P 7100 6600
+F 0 "C7" H 7215 6646 50  0000 L CNN
+F 1 "0.1uF" H 7215 6555 50  0000 L CNN
+F 2 "Capacitor_SMD:C_0805_2012Metric" H 7138 6450 50  0001 C CNN
+F 3 "~" H 7100 6600 50  0001 C CNN
+	1    7100 6600
+	1    0    0    -1
+$EndComp
+Wire Wire Line
+	6200 7150 7100 7150
+Wire Wire Line
+	7100 7150 7100 6750
+Connection ~ 6200 7150
+Wire Wire Line
+	6200 7150 6200 7000
+Wire Wire Line
+	7100 6450 7100 6000
+Wire Wire Line
+	7100 6000 6200 6000
 $EndSCHEMATC

Commit message: Swap audio jacks out
Parts:
- removed J4: AudioJack3, Connector_Audio:Jack_3.5mm_CUI_SJ-3523-SMT_Horizontal, symbol Connector:AudioJack3
- added J4, J8: Conn_Coaxial, td-io:CUI_RCJ-01X, symbol Connector:Conn_Coaxial
- J7: footprint td-io:DF1BZ-34DP-2.5DSA -> td-io:DF1BZ-34DP-2.5DS
Connections:
- wire segments 271 -> 275
Changed lines of the file:
@@
 speaker+
-$Comp
-L Connector:AudioJack3 J4
-U 1 1 6008792C
-P 800 8750
-F 0 "J4" H 782 9075 50  0000 C CNN
-F 1 "AudioJack3" H 782 8984 50  0000 C CNN
-F 2 "Connector_Audio:Jack_3.5mm_CUI_SJ-3523-SMT_Horizontal" H 800 8750 50  0001 C CNN
-F 3 "~" H 800 8750 50  0001 C CNN
-	1    800  8750
-	1    0    0    -1
-$EndComp
-Wire Wire Line
-	1000 8650 1300 8650
 $Comp
 L power:GND #PWR0123
 U 1 1 6008B983
-P 1150 8850
-F 0 "#PWR0123" H 1150 8600 50  0001 C CNN
-F 1 "GND" H 1155 8677 50  0000 C CNN
-F 2 "" H 1150 8850 50  0001 C CNN
-F 3 "" H 1150 8850 50  0001 C CNN
-	1    1150 8850
-	1    0    0    -1
-$EndComp
-Wire Wire Line
-	1150 8850 1000 8850
+P 1150 9200
+F 0 "#PWR0123" H 1150 8950 50  0001 C CNN
+F 1 "GND" H 1155 9027 50  0000 C CNN
+F 2 "" H 1150 9200 50  0001 C CNN
+F 3 "" H 1150 9200 50  0001 C CNN
+	1    1150 9200
+	1    0    0    -1
+$EndComp
 Connection ~ 15050 1400
 $Comp
@@
 $EndComp
 Wire Wire Line
-	13050 2700 13050 2850
+	13050 2700 13050 2750
 Wire Wire Line
 	12400 2500 12750 2500
@@
 	0    -1   -1   0
 $EndComp
-Wire Wire Line
-	13050 2200 13500 2200
 Connection ~ 13050 2200
 Wire Wire Line
@@
 F 0 "J7" H 5200 5267 50  0000 C CNN
 F 1 "Conn_02x17_Odd_Even" H 5200 5176 50  0000 C CNN
-F 2 "td-io:DF1BZ-34DP-2.5DSA" H 5150 4250 50  0001 C CNN
+F 2 "td-io:DF1BZ-34DP-2.5DS" H 5150 4250 50  0001 C CNN
 F 3 "~" H 5150 4250 50  0001 C CNN
 	1    5150 4250
@@
 	0    1    1    0
 $EndComp
-Wire Wire Line
-	1000 8750 1300 8750
-Wire Wire Line
-	1300 8750 1300 9050
 $Comp
 L Device:R R25
@@
 Wire Wire Line
 	7100 6000 6200 6000
+$Comp
+L Connector:Conn_Coaxial J4
+U 1 1 6022183D
+P 650 8650
+F 0 "J4" H 750 8532 50  0000 L CNN
+F 1 "Conn_Coaxial" H 750 8623 50  0000 L CNN
+F 2 "td-io:CUI_RCJ-01X" H 650 8650 50  0001 C CNN
+F 3 " ~" H 650 8650 50  0001 C CNN
+	1    650  8650
+	-1   0    0    1
+$EndComp
+$Comp
+L Connector:Conn_Coaxial J8
+U 1 1 60222C27
+P 650 9050
+F 0 "J8" H 750 8932 50  0000 L CNN
+F 1 "Conn_Coaxial" H 750 9023 50  0000 L CNN
+F 2 "td-io:CUI_RCJ-01X" H 650 9050 50  0001 C CNN
+F 3 " ~" H 650 9050 50  0001 C CNN
+	1    650  9050
+	-1   0    0    1
+$EndComp
+Wire Wire Line
+	850  8650 1300 8650
+Wire Wire Line
+	1300 9050 850  9050
+Wire Wire Line
+	1150 9200 1150 8850
+Wire Wire Line
+	1150 8850 650  8850
+Wire Wire Line
+	1150 8850 1150 8450
+Wire Wire Line
+	1150 8450 650  8450
+Connection ~ 1150 8850
+Wire Wire Line
+	13050 2750 13500 2750
+Wire Wire Line
+	13500 2750 13500 2200
+Connection ~ 13050 2750
+Wire Wire Line
+	13050 2750 13050 2850
 $EndSCHEMATC

Commit message: Add alternative power supply
Parts:
- removed U8, U9: 74LV166, Package_SO:SOIC-16_3.9x9.9mm_P1.27mm, symbol 74xx:74LS166
- added C?: 0.1uF, Capacitor_SMD:C_0805_2012Metric, symbol Device:C
- added C? (x2): 100uF, Capacitor_SMD:C_1206_3216Metric, symbol Device:C
- added C?: 1uF, Capacitor_SMD:C_0805_2012Metric, symbol Device:C
- added L?: 1uH, Inductor_SMD:L_7.3x7.3_H3.5, symbol Device:L
- added R? (x24): 10k, Resistor_SMD:R_0805_2012Metric, symbol Device:R
- added R?: 90k, Resistor_SMD:R_0805_2012Metric, symbol Device:R
- added R?: 20k, Resistor_SMD:R_0805_2012Metric, symbol Device:R
- added R?: 51k, symbol Device:R
- added R?: 160k, symbol Device:R
- added U? (x2): 74LV166, Package_SO:SOIC-16_3.9x9.9mm_P1.27mm, symbol 74xx:74LS166
- added U?: TPS568230, Package_DFN_QFN:VQFN-20-1EP_3x3mm_P0.45mm_EP1.55x1.55mm_ThermalVias, symbol td-io:TPS568230
- U5: value AD813 -> AT24CS01-SSHM
- renumbered U7 to U11
Connections:
- net +3V3: now also R?.1, R?.1, R?.1, R?.1, R?.1, R?.1, R?.1, R?.1, R?.1, R?.1, R?.1, R?.1, R?.1, R?.1, R?.1, R?.1, R?.1, R?.1, R?.1, R?.1, R?.1, R?.1, R?.1, R?.1, U?.16 (VCC), U?.16 (VCC); no longer J6.2 (Pin_2)
- net +5V: now also C?.1, U?.12 (EN), U?.2 (VIN), U?.3 (VIN), U?.4 (VIN), U?.5 (VIN)
- net GND: now also U6.1 (Ds), C?.2, C?.2, C?.2, R?.2, R?.2, U?.13 (AGND), U?.15 (PE), U?.15 (PE), U?.18 (GND), U?.21 (GND), U?.6 (CE), U?.6 (CE), U?.7 (GND), U?.8 (GND), U?.8 (GND), U?.8 (GND)
- net sr_clk: now also U?.7 (Clk), U?.7 (Clk)
- net sr_clr: now also U?.9 (Clr), U?.9 (Clr)
- net at U6.10 (E): now also R?.2
- net at U6.11 (F): now also R?.2
- net at U6.12 (G): now also R?.2
- net at U6.13 (Qh): now also U?.1 (Ds)
- net at U6.14 (H): now also R?.2
- net at U6.2 (A): now also R?.2
- net at U6.3 (B): now also R?.2
- net at U6.4 (C): now also R?.2
- net at U6.5 (D): now also R?.2
- new net: R?.2, U?.10 (E) (x2)
- new net: R?.2, U?.11 (F) (x2)
- new net: R?.2, U?.12 (G) (x2)
- new net: U?.1 (Ds), U?.13 (Qh)
- new net: R?.2, U?.14 (H) (x2)
- new net: R?.2, U?.2 (A) (x2)
- new net: R?.2, U?.3 (B) (x2)
- new net: R?.2, U?.4 (C) (x2)
- new net: R?.2, U?.5 (D) (x2)
- new net: C?.2, U?.1 (VBST)
- new net: R?.1, R?.2, U?.14 (FB)
- new net: R?.1, R?.2, U?.15 (MODE)
- new net: C?.1, R?.1, U?.17 (VCC)
- new net: C?.1, L?.1, U?.19 (SW), U?.20 (SW), U?.6 (SW)
- new net +3.3VP: C?.1, J6.2 (Pin_2), L?.2, R?.1
- no-connect marks 36 -> 38
Other:
- moved on the sheet: C12, C13, C14, C15, C16, C17, C18, D1, D2, J6, L1, Q1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

Commit message: Add JVS chaining support
Parts:
- removed C12, C13, C14: 10uF, Capacitor_SMD:C_0805_2012Metric, symbol Device:C
- removed C15: 750pF, Capacitor_SMD:C_0805_2012Metric, symbol Device:C
- removed C16: 100uF, Capacitor_SMD:CP_Elec_5x5.3, symbol Device:CP
- removed C17: 1uF, Capacitor_SMD:C_0805_2012Metric, symbol Device:C
- removed C18: 1000pF, Capacitor_SMD:C_0805_2012Metric, symbol Device:C
- removed D1: SL44-E3/57T, Diode_SMD:D_SMC, symbol Device:D_Schottky
- removed L1: 0.1mH, Inductor_THT:L_Toroid_Horizontal_D32.5mm_P30.00mm_Bourns_2300, symbol Device:L
- removed Q1: Si7141DP, Package_SO:PowerPAK_SO-8_Single, symbol Transistor_FET:Si7141DP
- removed R20: 15.4k, Resistor_SMD:R_0805_2012Metric, symbol Device:R
- removed R21: 2.94k, Resistor_SMD:R_0805_2012Metric, symbol Device:R
- removed R22: 0.01, Resistor_SMD:R_0805_2012Metric, symbol Device:R
- removed R23: 10k, Resistor_SMD:R_0805_2012Metric, symbol Device:R
- removed R24: 6.04k, Resistor_SMD:R_0805_2012Metric, symbol Device:R
- removed U11: LM25085MM, Package_SO:MSOP-8_3x3mm_P0.65mm, symbol Regulator_Switching:LM25085MM
- removed U2: ST485EB, Package_SO:SOIC-8_3.9x4.9mm_P1.27mm, symbol Interface_UART:ST485EBDR
- added D1: BAV99S, Package_TO_SOT_SMD:SOT-363_SC-70-6, symbol Diode:BAV99S
- added H1, H2, H3, H4: MountingHole_Pad, MountingHole:MountingHole_3.2mm_M3_Pad_Via, symbol Mechanical:MountingHole_Pad
- added Q1: FDS6930B, Package_SO:SOIC-8_3.9x4.9mm_P1.27mm, symbol Transistor_FET:FDS6930B
- added R50, R51, R52, R54: 10k, symbol Device:R
- added R53: 20k, symbol Device:R
- added R55: R, symbol Device:R
- added U11: TL081, symbol Amplifier_Operational:TL081
- added U12: CPC1017N, Package_SO:SOP-4_3.8x4.1mm_P2.54mm, symbol Relay_SolidState:CPC1017N
- added U2: SP3481CN, Package_SO:SOIC-8_3.9x4.9mm_P1.27mm, symbol Interface_UART:SP3481CN
- Q2, Q3: value FDS6930A -> FDS6930B; symbol Transistor_FET:FDS6930A -> Transistor_FET:FDS6930B
- Q2: value FDS6930A -> FDS6930B
- R1, R2, R3, R4: value R -> 20k
- R20, R21: renamed from R?; footprint (none) -> Resistor_SMD:R_0805_2012Metric
- RV1: footprint Potentiometer_THT:Potentiometer_Alps_RK09K_Single_Vertical -> Potentiometer_THT:Potentiometer_Bourns_PTV09A-1_Single_Vertical
- gave numbers to parts that had none: 34
Connections:
- net +3V3: now also C3.1, U2.8 (VCC)
- net +5V: now also R51.1, U11.7 (V+); no longer C3.1
- net GND: now also D1.5 (K4), H1.1, H2.1, H3.1, H4.1, Q1.1 (S1), R50.2, R52.2, U11.3 (+), U11.4 (V-), U2.5 (GND)
- net c1: now also R31.2, U6.2 (A)
- net c2: now also R30.2, U6.3 (B)
- net jvs_de: now also U2.3 (DE)
- net jvs_re: now also U2.2 (~RE~)
- net jvs_rx: now also U2.1 (RO)
- net jvs_tx: now also U2.4 (DI)
- net p1_1: now also R37.2, U8.10 (E)
- net p1_2: now also R35.2, U8.12 (G)
- net p1_3: now also R49.2, U9.2 (A)
- net p1_4: now also R47.2, U9.4 (C)
- net p1_5: now also R45.2, U9.10 (E)
- net p1_6: now also R43.2, U9.12 (G)
- net p1down: now also R23.2, U6.12 (G)
- net p1left: now also R41.2, U8.2 (A)
- net p1right: now also R39.2, U8.4 (C)
- net p1start: now also R29.2, U6.4 (C)
- net p1up: now also R27.2, U6.10 (E)
- net p2_1: now also R36.2, U8.11 (F)
- net p2_2: now also R34.2, U8.14 (H)
- net p2_3: now also R48.2, U9.3 (B)
- net p2_4: now also R46.2, U9.5 (D)
- net p2_5: now also R44.2, U9.11 (F)
- net p2_6: now also R42.2, U9.14 (H)
- net p2down: now also R22.2, U6.14 (H)
- net p2left: now also R40.2, U8.3 (B)
- net p2right: now also R38.2, U8.5 (D)
- net p2start: now also R28.2, U6.5 (D)
- net p2up: now also R24.2, U6.11 (F)
- net sr_data: now also U9.13 (Qh)
- net at J1.1 (VBUS): now also R51.2, R53.2
- net at J1.2 (D-), J2.2 (D-): now also U12.4, U2.6 (A); no longer R5.2
- net at J1.3 (D+), J2.3 (D+), R5.1: now also R55.1, U2.7 (B)
- net at J2.1 (VBUS): now also Q1.5 (D2), Q1.6 (D2), Q1.7 (D1), Q1.8 (D1)
- net sense_0v: now reaches U10.17 (GPIO13)
- net sense_0v: now also Q1.2 (G1), R50.1
- net sense_2.5v: now reaches U10.19 (GPIO14)
- net sense_2.5v: now also Q1.4 (G2), R52.1
- net termination: now reaches U10.20 (GPIO15)
- net termination: now also U12.2
- net sense_in: now reaches U10.31 (GPIO26_ADC0)
- net sense_in: now also R54.1, U11.6
- net SW: now reaches C11.1, L1.1, U7.19 (SW), U7.20 (SW), U7.6 (SW)
- net p1select: no longer names the net of J3.26 (Unused)
- net p2select: no longer names the net of J3.d (Unused)
- new net: R5.2, U12.3
- new net: R53.1, R54.2, U11.2 (-)
- new net: R55.2, U12.1
- new net: D1.1 (A1), Q1.3 (S2)
- new net: D1.2 (K2), D1.4 (A3)
- no-connect marks 38 -> 53
Other:
- note removed: "consider Si7149DP"
- moved on the sheet: C1, C10, C11, C12, C2, C3, C4, C8, C9, J1, J2, J4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
