File: td-io.sch (KiCad schematic (older format))
At the start: 107 parts, among them J1 USB_A, J2 USB_B, J3 JAMMA_Edge, J4 Conn_Coaxial, J5 DB15_Female_HighDensity, J6 Conn_02x04_Top_Bottom, J7 Conn_02x17_Odd_Even, J8 Conn_Coaxial, Q1 FDS6930B, Q2 FDS6930B, Q3 FDS6930B, SW1 SW_DIP_x02, U1 LM4950TS, U10 Pico, U11 TL081, U12 CPC1017N, U13 74LS165, U2 SP3481CN, U3 AD813, U4 74LS86, U5 AT24CS01-SSHM, U6 74LS165, U7 TPS568230, U8 74LS165, U9 74LS165

Commit message: Swap to ADA4891-3.
Parts:
- U3: value AD813 -> ADA4891-3; symbol Amplifier_Video:AD813 -> td-io:ADA4891-3
Changed lines of the file:
@@
 Connection ~ 10700 10050
 $Comp
-L Amplifier_Video:AD813 U3
+L td-io:ADA4891-3 U3
 U 1 1 600EAC98
 P 8100 5900
 F 0 "U3" H 8100 6267 50  0000 C CNN
-F 1 "AD813" H 8100 6176 50  0000 C CNN
+F 1 "ADA4891-3" H 8100 6176 50  0000 C CNN
 F 2 "Package_SO:SOIC-14_3.9x8.7mm_P1.27mm" H 8100 5900 50  0001 C CNN
-F 3 "https://www.analog.com/media/en/technical-documentation/data-sheets/AD813.pdf" H 8100 5900 50  0001 C CNN
+F 3 "https://www.analog.com/media/en/technical-documentation/data-sheets/ADA4891-1_4891-2_4891-3_4891-4.PDF" H 8100 5900 50  0001 C CNN
 	1    8100 5900
 	1    0    0    -1
 $EndComp
 $Comp
-L Amplifier_Video:AD813 U3
+L td-io:ADA4891-3 U3
 U 4 1 600EF901
 P 10550 6000
 F 0 "U3" H 10508 6046 50  0000 L CNN
-F 1 "AD813" H 10508 5955 50  0000 L CNN
+F 1 "ADA4891-3" H 10508 5955 50  0000 L CNN
 F 2 "Package_SO:SOIC-14_3.9x8.7mm_P1.27mm" H 10550 6000 50  0001 C CNN
-F 3 "https://www.analog.com/media/en/technical-documentation/data-sheets/AD813.pdf" H 10550 6000 50  0001 C CNN
+F 3 "https://www.analog.com/media/en/technical-documentation/data-sheets/ADA4891-1_4891-2_4891-3_4891-4.PDF" H 10550 6000 50  0001 C CNN
 	4    10550 6000
 	1    0    0    -1
@@
 vga_red
 $Comp
-L Amplifier_Video:AD813 U3
+L td-io:ADA4891-3 U3
 U 2 1 60095C91
 P 8100 7450
 F 0 "U3" H 8100 7817 50  0000 C CNN
-F 1 "AD813" H 8100 7726 50  0000 C CNN
+F 1 "ADA4891-3" H 8100 7726 50  0000 C CNN
 F 2 "Package_SO:SOIC-14_3.9x8.7mm_P1.27mm" H 8100 7450 50  0001 C CNN
-F 3 "https://www.analog.com/media/en/technical-documentation/data-sheets/AD813.pdf" H 8100 7450 50  0001 C CNN
+F 3 "https://www.analog.com/media/en/technical-documentation/data-sheets/ADA4891-1_4891-2_4891-3_4891-4.PDF" H 8100 7450 50  0001 C CNN
 	2    8100 7450
 	1    0    0    -1
@@
 vga_green
 $Comp
-L Amplifier_Video:AD813 U3
+L td-io:ADA4891-3 U3
 U 3 1 6009DE48
 P 8050 9000
 F 0 "U3" H 8050 9367 50  0000 C CNN
-F 1 "AD813" H 8050 9276 50  0000 C CNN
+F 1 "ADA4891-3" H 8050 9276 50  0000 C CNN
 F 2 "Package_SO:SOIC-14_3.9x8.7mm_P1.27mm" H 8050 9000 50  0001 C CNN
-F 3 "https://www.analog.com/media/en/technical-documentation/data-sheets/AD813.pdf" H 8050 9000 50  0001 C CNN
+F 3 "https://www.analog.com/media/en/technical-documentation/data-sheets/ADA4891-1_4891-2_4891-3_4891-4.PDF" H 8050 9000 50  0001 C CNN
 	3    8050 9000
 	1    0    0    -1
@@
 Text Label 3000 2350 0    50   ~ 0
 jamma_sync
-Text Label 6900 10350 0    50   ~ 0
+Text Label 11650 7700 0    50   ~ 0
 jamma_sync
 $Comp

Commit message: Switch to class D amp
Parts:
- removed R2, R3, R4: 20k, Resistor_SMD:R_0805_2012Metric, symbol Device:R
- removed RV1: 10k Audio, Potentiometer_THT:Potentiometer_Bourns_PTV09A-1_Single_Vertical, symbol Device:R_POT
- removed U1: LM4950TS, Package_TO_SOT_SMD:TO-263-9_TabPin5, symbol Amplifier_Audio:LM4950TS
- added C17, C18: 100uF, Capacitor_SMD:C_1206_3216Metric, symbol Device:C
- added C19, C20, C21, C22, C23: 1uF, Capacitor_SMD:C_0805_2012Metric, symbol Device:C
- added C24, C25, C26, C27: 2.2uF, Capacitor_SMD:C_0805_2012Metric, symbol Device:C
- added J9: Conn_01x04_Male, Connector_JST:JST_EH_B4B-EH-A_1x04_P2.50mm_Vertical, symbol Connector:Conn_01x04_Male
- added L2, L3, L4, L5: 15uH, Inductor_SMD:L_7.3x7.3_H4.5, symbol Device:L
- added RV1: R_POT_Dual, Potentiometer_THT:Potentiometer_Alpha_RD902F-40-00D_Dual_Vertical_CircularHoles, symbol Device:R_POT_Dual
- added U1: TPA3138D2, Package_SO:HTSSOP-28-1EP_4.4x9.7mm_P0.65mm_EP2.85x5.4mm_ThermalVias, symbol td-io:TPA3138D2
- C1: value 0.1uF -> 1uF
- C4: value 10uF -> 1uF
- R1: value 20k -> 10k
Connections:
- net +12V: now also R1.2, C17.1, C18.1, U1.15 (PVCC), U1.16 (PVCC), U1.27 (PVCC), U1.28 (PVCC), U1.7 (AVCC); no longer C1.1
- net GND: now also C1.1, C4.1, C17.2, C18.2, C21.1, C24.2, C25.2, C26.2, C27.2, RV1.3, RV1.6, U1.10 (PLIMIT), U1.14 (GND), U1.19 (GND), U1.24 (GND), U1.29 (PAD), U1.5 (GAIN_SEL), U1.6 (MODE_SEL), U1.8 (GND); no longer C1.2, C4.2
- net speaker+: now also C19.1, C24.1, J9.4 (Pin_4), L2.2
- net speaker-: now also C22.1, C25.1, J9.2 (Pin_2), L3.2; no longer R1.2
- net at R1.1: now also U1.2 (~SD2/FAULT)
- net at R25.1: now also RV1.1; no longer R26.1
- new net: C4.2, U1.11 (RINN)
- new net: RV1.5, U1.12 (RINP)
- new net: C23.2, U1.17 (BSPR)
- new net: L5.1, U1.18 (OUTPR)
- new net: L4.1, U1.20 (OUTNR)
- new net: C20.2, U1.21 (BSNR)
- new net: C22.2, U1.22 (BSNL)
- new net: L3.1, U1.23 (OUTNL)
- new net: L2.1, U1.25 (OUTPL)
- new net: C19.2, U1.26 (BSPL)
- new net: RV1.2, U1.3 (LINP)
- new net: C1.2, U1.4 (LINN)
- new net: C21.2, U1.9 (GVDD)
- new net: R26.1, RV1.4
- new net speaker_r+: C23.1, C27.1, J9.1 (Pin_1), L5.2
- new net speaker_r-: C20.1, C26.1, J9.3 (Pin_3), L4.2
- no-connect marks 55 -> 57
Other:
- note removed: "consider ac coupling"
- moved on the sheet: C10, C11, C12, C13, C14, C15, C16, C2, C3, C5, C6, C7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

Commit message: more layout
Parts:
- added SW2: SW_DIP_x01, Button_Switch_SMD:SW_DIP_SPSTx01_Slide_Omron_A6S-110x_W8.9mm_P2.54mm, symbol Switch:SW_DIP_x01
- Q2, Q3: value FDS6930B -> ZXMS6004DN8
- RV1: footprint Potentiometer_THT:Potentiometer_Alpha_RD902F-40-00D_Dual_Vertical_CircularHoles -> td-io:PTV112-4420A-A503; Digikey (none) -> PTV112-4420A-A503-ND
Connections:
- net at RV1.5, U1.12 (RINP): now also SW2.1
- net at RV1.2, U1.3 (LINP): now also SW2.2
- net -5V: no longer names the net of J3.5 (-5V)
- net -5V: no longer J3.E (-5V)
- no-connect marks 57 -> 59
Changed lines of the file:
@@
 Connection ~ 15600 3750
 $Comp
-L power:-5V #PWR0105
-U 1 1 6002FF85
-P 13100 3950
-F 0 "#PWR0105" H 13100 4050 50  0001 C CNN
-F 1 "-5V" H 13115 4123 50  0000 C CNN
-F 2 "" H 13100 3950 50  0001 C CNN
-F 3 "" H 13100 3950 50  0001 C CNN
-	1    13100 3950
-	-1   0    0    1
-$EndComp
-Wire Wire Line
-	13100 3950 13800 3950
-$Comp
-L power:-5V #PWR0106
-U 1 1 600316B6
-P 16100 3950
-F 0 "#PWR0106" H 16100 4050 50  0001 C CNN
-F 1 "-5V" H 16115 4123 50  0000 C CNN
-F 2 "" H 16100 3950 50  0001 C CNN
-F 3 "" H 16100 3950 50  0001 C CNN
-	1    16100 3950
-	-1   0    0    1
-$EndComp
-Wire Wire Line
-	15450 3950 16100 3950
-$Comp
 L power:+12V #PWR0107
 U 1 1 60032807
@@
 F 0 "RV1" V 2804 4213 50  0000 R CNN
 F 1 "R_POT_Dual" V 2895 4213 50  0000 R CNN
-F 2 "Potentiometer_THT:Potentiometer_Alpha_RD902F-40-00D_Dual_Vertical_CircularHoles" H 3100 4325 50  0001 C CNN
+F 2 "td-io:PTV112-4420A-A503" H 3100 4325 50  0001 C CNN
 F 3 "~" H 3100 4325 50  0001 C CNN
+F 4 "PTV112-4420A-A503-ND" V 2850 4400 50  0001 C CNN "Digikey"
 	1    2850 4400
 	0    1    1    0
@@
 	2950 4150 2950 4550
 Wire Wire Line
-	2950 4550 3500 4550
+	2950 4550 3050 4550
 $Comp
 L Device:C C1
@@
 	2950 4650 2950 4950
 Wire Wire Line
-	2950 4950 3500 4950
+	2950 4950 3150 4950
 Wire Wire Line
 	3500 4650 3000 4650
@@
 P 7450 7250
 F 0 "Q3" H 7654 7296 50  0000 L CNN
-F 1 "FDS6930B" H 7654 7205 50  0000 L CNN
+F 1 "ZXMS6004DN8" H 7654 7205 50  0000 L CNN
 F 2 "Package_SO:SOIC-8_3.9x4.9mm_P1.27mm" H 7650 7175 50  0001 L CIN
 F 3 "http://www.onsemi.com/pub/Collateral/FDS6930B-D.PDF" H 7450 7250 50  0001 L CNN
@@
 P 7150 6500
 F 0 "Q2" H 7354 6546 50  0000 L CNN
-F 1 "FDS6930B" H 7354 6455 50  0000 L CNN
+F 1 "ZXMS6004DN8" H 7354 6455 50  0000 L CNN
 F 2 "Package_SO:SOIC-8_3.9x4.9mm_P1.27mm" H 7350 6425 50  0001 L CIN
 F 3 "http://www.onsemi.com/pub/Collateral/FDS6930B-D.PDF" H 7150 6500 50  0001 L CNN
@@
 P 8550 7300
 F 0 "Q3" H 8754 7346 50  0000 L CNN
-F 1 "FDS6930B" H 8754 7255 50  0000 L CNN
+F 1 "ZXMS6004DN8" H 8754 7255 50  0000 L CNN
 F 2 "Package_SO:SOIC-8_3.9x4.9mm_P1.27mm" H 8750 7225 50  0001 L CIN
 F 3 "http://www.onsemi.com/pub/Collateral/FDS6930B-D.PDF" H 8550 7300 50  0001 L CNN
@@
 P 8300 6500
 F 0 "Q2" H 8504 6546 50  0000 L CNN
-F 1 "FDS6930B" H 8504 6455 50  0000 L CNN
+F 1 "ZXMS6004DN8" H 8504 6455 50  0000 L CNN
 F 2 "Package_SO:SOIC-8_3.9x4.9mm_P1.27mm" H 8500 6425 50  0001 L CIN
 F 3 "http://www.onsemi.com/pub/Collateral/FDS6930B-D.PDF" H 8300 6500 50  0001 L CNN
@@
 NoConn ~ 13800 8500
 NoConn ~ 13800 8600
+$Comp
+L Switch:SW_DIP_x01 SW2
+U 1 1 603AAE71
+P 2100 3400
+F 0 "SW2" H 2100 3667 50  0000 C CNN
+F 1 "SW_DIP_x01" H 2100 3576 50  0000 C CNN
+F 2 "Button_Switch_SMD:SW_DIP_SPSTx01_Slide_Omron_A6S-110x_W8.9mm_P2.54mm" H 2100 3400 50  0001 C CNN
+F 3 "~" H 2100 3400 50  0001 C CNN
+	1    2100 3400
+	1    0    0    -1
+$EndComp
+Wire Wire Line
+	3050 4550 3050 3850
+Wire Wire Line
+	3050 3850 2400 3850
+Wire Wire Line
+	2400 3850 2400 3400
+Connection ~ 3050 4550
+Wire Wire Line
+	3050 4550 3500 4550
+Wire Wire Line
+	3150 4950 3150 4000
+Wire Wire Line
+	3150 4000 2900 4000
+Wire Wire Line
+	2900 4000 2900 3900
+Wire Wire Line
+	2900 3900 2450 3900
+Wire Wire Line
+	2450 3900 2450 3550
+Wire Wire Line
+	2450 3550 1800 3550
+Wire Wire Line
+	1800 3550 1800 3400
+Connection ~ 3150 4950
+Wire Wire Line
+	3150 4950 3500 4950
+NoConn ~ 15450 3950
+NoConn ~ 13800 3950
 $EndSCHEMATC

Commit message: BOM updates
Parts:
- C1, C10, C19, C2, C20, C21, C22, C23, C4, C8: Digikey (none) -> 1276-2926-1-ND
- C11, C13, C14, C15, C16, C3, C5, C6, C7: Digikey (none) -> 1276-2444-1-ND
- C12, C9: Digikey (none) -> 1276-1782-1-ND
- C17, C18: value 100uF -> 100uF 16V; Digikey (none) -> 565-4527-1-ND
- C24, C25, C26, C27: Digikey (none) -> 1276-2954-1-ND
- D1: Digikey (none) -> 1727-4042-1-ND
- D2: Digikey (none) -> 1727-2901-1-ND
- J1: Digikey (none) -> WM14667-ND
- J2: Digikey (none) -> ED2982-ND
- J4: Digikey (none) -> CP-1402-ND
- J5: footprint Connector_Dsub:DSUB-15-HD_Female_Horizontal_P2.29x1.98mm_EdgePinOffset3.03mm_Housed_MountingHolesOffset4.94mm -> td-io:DSUB-15-HD_Female_Horizontal_P2.29x2.5mm_EdgePinOffset8.35mm_Housed_MountingHolesOffset10.89mm; Digikey (none) -> L77HDE15SD1CH4F-ND
- J6: Digikey (none) -> 455-2365-ND
- J7: Digikey (none) -> H11039-ND
- J8: Digikey (none) -> CP-1401-ND
- J9: Digikey (none) -> 455-4179-ND
- Q1, Q2, Q3: Digikey (none) -> ZXMS6004DN8-13DICT-ND
- R1, R22, R23, R24, R27, R28, R29, R30, R31, R34, R35, R36, R37, R38, R39, R40, R41, R42, R43, R44, R45, R46, R47, R48, R49, R50, R51, R52, R54, R56, R57, R58, R6, R7: Digikey (none) -> 311-10.0KCRCT-ND
- R10, R8, R9: Digikey (none) -> 311-75.0CRCT-ND
- R11, R12, R13: Digikey (none) -> 311-100CRCT-ND
- R14, R15, R16, R25, R26: Digikey (none) -> 311-1.00KCRCT-ND
- R17, R18, R19: value R -> 75; Digikey (none) -> 311-75.0CRCT-ND
- R20: Digikey (none) -> 311-158KCRTR-ND
- R21: Digikey (none) -> 311-51.1KCRCT-ND
- R32: value 90k -> 91k; Digikey (none) -> 311-91.0KCRCT-ND
- R33, R53: Digikey (none) -> 311-20.0KCRCT-ND
- R5: Digikey (none) -> 311-120CRCT-ND
- R55: value R -> 1k; Digikey (none) -> 311-1.00KCRCT-ND
- SW1: Digikey (none) -> SW1190-ND
- SW2: Digikey (none) -> Z5187-ND
- U1: Digikey (none) -> 296-50219-ND
- U10: footprint MCU_RaspberryPi_and_Boards:RPi_Pico_SMD_TH -> td-io:RPi_Pico_SMD; Digikey (none) -> 2648-SC0915CT-ND
- U11: Digikey (none) -> 296-15001-1-ND
- U12: Digikey (none) -> CLA153-ND
- U13, U6, U8, U9: Digikey (none) -> 296-SN74LV165ADRG3CT-ND
- U2: value SP3481CN -> ISL3175EIBZ-T; Digikey (none) -> ISL3175EIBZ-TCT-ND
- U3: Digikey (none) -> ADA4891-3ARZ-ND
- U4: Digikey (none) -> 1727-3464-ND
- U5: Digikey (none) -> AT24CS01-SSHM-TCT-ND
- U7: Digikey (none) -> 296-TPS568230RJERCT-ND

Commit message: Add todo
Other:
- note added: "todo:\nnew footprint for RCA jacks\nsmaller ground pad tor tpa3138d2\nsmaller ground pad for tps568230\nfix pin 11/14 swap on VGA jack\nfix DISABLE on ada4891\nadd additional input capacitance on tps568230\nconnect power/ground to xor gate\nmove AC coupling on audio input to after volume pot\nconnect boost caps on tpa3138 before inductor\nincrease tpa3138 output caps' voltage rating for reduced t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"
Changed lines of the file:
@@
 NoConn ~ 15450 3950
 NoConn ~ 13800 3950
+Text Notes 8700 9100 0    50   ~ 0
+todo:\nnew footprint for RCA jacks\nsmaller ground pad tor tpa3138d2\nsmaller ground pad for tps568230\nfix pin 11/14 swap on VGA jack\nfix DISABLE on ada4891\nadd additional input capacitance on tps568230\nconnect power/ground to xor gate\nmove AC coupling on audio input to after volume pot\nconnect boost caps on tpa3138 before inductor\nincrease tpa3138 output caps' voltage rating for reduced thd\nmake JST-SH footprint\nmove stereo connector farther away from caps\nchange vga amp gain
 $EndSCHEMATC
