File: td-io.sch (KiCad schematic (older format))
At the start: 121 parts, among them J1 USB_A, J2 USB_B, J3 JAMMA_Edge, J4 Conn_Coaxial, J5 DB15_Female_HighDensity, J6 Conn_02x04_Top_Bottom, J7 Conn_02x17_Odd_Even, J8 Conn_Coaxial, J9 Conn_01x04_Male, Q1 FDS6930B, Q2 ZXMS6004DN8, Q3 ZXMS6004DN8, SW1 SW_DIP_x02, SW2 SW_DIP_x01, U1 TPA3138D2, U10 Pico, U11 TL081, U12 CPC1017N, U13 74LS165, U2 ISL3175EIBZ-T, U3 ADA4891-3, U4 74LS86, U5 AT24CS01-SSHM, U6 74LS165, U7 TPS568230, U8 74LS165, U9 74LS165

Commit message: changes
Parts:
- removed J4, J8: Conn_Coaxial, td-io:CUI_RCJ-01X, symbol Connector:Conn_Coaxial
- removed J5: DB15_Female_HighDensity, td-io:DSUB-15-HD_Female_Horizontal_P2.29x2.5mm_EdgePinOffset8.35mm_Housed_MountingHolesOffset10.89mm, symbol Connector:DB15_Female_HighDensity
- removed R53: 20k, Resistor_SMD:R_0805_2012Metric, symbol Device:R
- removed R54: 10k, Resistor_SMD:R_0805_2012Metric, symbol Device:R
- removed U11: TL081, Package_SO:SOIC-8_3.9x4.9mm_P1.27mm, symbol Amplifier_Operational:TL081
- added C28, C30, C31: 3.3uF, Capacitor_SMD:C_0805_2012Metric, symbol Device:C
- added C29, C32: 0.1uF, Capacitor_SMD:C_0805_2012Metric, symbol Device:C
- added J4: Conn_Coaxial_x2, td-io:PJRAN2X1U01AUX, symbol Connector:Conn_Coaxial_x2
- added J5: DB15_Female_HighDensity_MountingHoles, td-io:DSUB-15-HD_Female_Horizontal_P2.29x2.5mm_EdgePinOffset8.35mm_Housed_MountingHolesOffset10.89mm, symbol Connector:DB15_Female_HighDensity_MountingHoles
- added R2: 400k, Resistor_SMD:R_0805_2012Metric, symbol Device:R
- added R3: 1k, Resistor_SMD:R_0805_2012Metric, symbol Device:R
- added R4: 10k, Resistor_SMD:R_0805_2012Metric, symbol Device:R
- added U11: LM2664M4, Package_TO_SOT_SMD:SOT-23-6, symbol td-io:LM2664M4
- added U14: TPS259620, Package_SO:SOIC-8-1EP_3.9x4.9mm_P1.27mm_EP2.41x3.3mm_ThermalVias, symbol td-io:TPS259631
- added U15: LM2903, Package_SO:SOIC-8_3.9x4.9mm_P1.27mm, symbol Comparator:LM2903
- added unit 3 of U4
- added unit 4 of U4
- added unit 5 of U4
- C12, C9: footprint Capacitor_SMD:C_1206_3216Metric -> Capacitor_SMD:C_1210_3225Metric
- C24, C25, C26, C27: footprint Capacitor_SMD:C_0805_2012Metric -> Capacitor_SMD:C_1210_3225Metric; Digikey 1276-2954-1-ND -> 1276-3362-1-ND
- J9: footprint Connector_JST:JST_EH_B4B-EH-A_1x04_P2.50mm_Vertical -> td-io:JST_SH_B4B-NH-A_1x04_P2.50mm_Vertical
- L1: value 1uH -> 1.5uH; footprint Inductor_SMD:L_7.3x7.3_H3.5 -> Inductor_SMD:L_Bourns_SRR1260; Digikey 2184-BMRA000606301R0MA1CT-ND -> SRR1260-1R5YTR-ND
- Q1: Digikey ZXMS6004DN8-13DICT-ND -> (none)
- R11, R12, R13: value 100 -> 330
- R20: value 160k -> 300k
- R21: value 51k -> 43k
- R25: value 1k -> 20k; Digikey 311-1.00KCRCT-ND -> (none)
- R26: value 1k -> 10k; Digikey 311-1.00KCRCT-ND -> (none)
- R52: value 10k -> 100
- U1: footprint Package_SO:HTSSOP-28-1EP_4.4x9.7mm_P0.65mm_EP2.85x5.4mm_ThermalVias -> td-io:HTSSOP-28-1EP_4.4x9.7mm_P0.65mm_tpa3138_ThermalVias
- U3: value ADA4891-3 -> ADA4861-3
- U7: footprint Package_DFN_QFN:VQFN-20-1EP_3x3mm_P0.45mm_EP1.55x1.55mm_ThermalVias -> td-io:RJE-20
Connections:
- net labels added: +5VL, -5V, l_in, r_in, sense_in_high, sense_in_low
- net labels removed: sense_in
- wire segments 457 -> 508
- no-connect marks 59 -> 57
Other:
- note added: "todo:\nmove stereo connector farther away from caps\ndifferent vga connector without text on it\nreposition connectors\n"
- note removed: "todo:\nnew footprint for RCA jacks\nsmaller ground pad tor tpa3138d2\nsmaller ground pad for tps568230\nfix pin 11/14 swap on VGA jack\nfix DISABLE on ada4891\nadd additional input capacitance on tps568230\nconnect power/ground to xor gate\nmove AC coupling on audio input to after volume pot\nconnect boost caps on tpa3138 before inductor\nincrease tpa3138 output caps' voltage rating for reduced t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"
- moved on the sheet: C2, C8, C9, L2, L3, L4, L5, R52, RV1

Commit message: change switch
Parts:
- removed SW2: SW_DIP_x01, Button_Switch_SMD:SW_DIP_SPSTx01_Slide_Omron_A6S-110x_W8.9mm_P2.54mm, symbol Switch:SW_DIP_x01
- added C33: 3.3uF, Capacitor_SMD:C_0805_2012Metric, symbol Device:C
- added C34, C35: 0.1uF, Capacitor_SMD:C_0805_2012Metric, symbol Device:C
- added C36, C37: 47uF 16V, Capacitor_SMD:C_1210_3225Metric, symbol Device:C
- added SW2: SW_DPDT_x2, Button_Switch_SMD:SW_DPDT_CK_JS202011JCQN, symbol Switch:SW_DPDT_x2
- C17, C18: value 100uF 16V -> 47uF 16V; footprint Capacitor_SMD:C_1206_3216Metric -> Capacitor_SMD:C_1210_3225Metric; Digikey 565-4527-1-ND -> 490-16309-1-ND
Connections:
- wire segments 508 -> 520
Other:
- moved on the sheet: C17, C18, C5, C7, H1, H2, H3, H4, J5, R6, R7, U4A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

Commit message: Move some tracks around
Parts:
- added J?: Conn_01x05_Male, Connector_JST:JST_XH_B5B-XH-A_1x05_P2.50mm_Vertical, symbol Connector:Conn_01x05_Male
Connections:
- net +3V3: now also J?.1 (Pin_1)
- net GND: now also J?.5 (Pin_5)
- net adc0: now reaches U10.31 (GPIO26_ADC0)
- net adc0: now also J?.2 (Pin_2)
- net adc1: now reaches U10.32 (GPIO27_ADC1)
- net adc1: now also J?.3 (Pin_3)
- net adc2: now reaches U10.34 (GPIO28_ADC2)
- net adc2: now also J?.4 (Pin_4)
- no-connect marks 57 -> 55
Other:
- moved on the sheet: Q1B

Commit message: add dc restoration and incrase schematic size
Parts:
- removed R10, R8: 75, Resistor_SMD:R_0805_2012Metric, symbol Device:R
- added C? (x3): 1uF, symbol Device:C
- added Q? (x3): 2N7002NXBKR, Package_TO_SOT_SMD:SOT-23, symbol Transistor_FET:2N7002
- added R? (x3): 10k, symbol Device:R
- added R? (x2): 75, Resistor_SMD:R_0805_2012Metric, symbol Device:R
- J8: renamed from J?; footprint Connector_JST:JST_XH_B5B-XH-A_1x05_P2.50mm_Vertical -> Connector_PinHeader_2.54mm:PinHeader_1x05_P2.54mm_Vertical
- Q1: value FDS6930B -> ZXMS6004DN8
Connections:
- net GND: now also Q?.2 (S), Q?.2 (S), Q?.2 (S), R?.1, R?.1, R?.2, R?.2, R?.2
- net vga_blue: now also C?.2, R?.2; no longer U3.10 (+)
- net vga_green: now also C?.2, R?.2; no longer U3.12 (+)
- net vga_red: now also C?.2; no longer U3.5 (+)
- new net: C?.1, Q?.3 (D), R?.1, U3.12 (+)
- new net: C?.1, Q?.3 (D), R?.1, U3.10 (+)
- new net: C?.1, Q?.3 (D), R?.1, U3.5 (+)
- new net blank: Q?.1 (G), Q?.1 (G), Q?.1 (G)
Other:
- moved on the sheet: C10, C11, C12, C17, C18, C28, C29, C30, C31, C33, C34, C35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

Commit message: more fixes
Parts:
- removed SW1: SW_DIP_x02, Button_Switch_SMD:SW_DIP_SPSTx02_Slide_Omron_A6S-210x_W8.9mm_P2.54mm, symbol Switch:SW_DIP_x02
- added SW1, SW2: SW_DPDT_x2, Button_Switch_SMD:SW_DPDT_CK_JS202011JCQN, symbol Switch:SW_DPDT_x2
- C28, C30, C31: Digikey (none) -> 1276-6461-1-ND
- C29: Digikey (none) -> 1276-2444-1-ND
- C33: Digikey 1276-2444-1-ND -> 1276-6461-1-ND
- C38, C39, C40: renamed from C?; footprint (none) -> Capacitor_SMD:C_0805_2012Metric; Digikey (none) -> 1276-2926-1-ND
- J4: Digikey (none) -> SC2534-ND
- J5: Digikey (none) -> Z13226-ND
- L1: footprint Inductor_SMD:L_Bourns_SRR1260 -> Inductor_SMD:L_Bourns_SRP7028A_7.3x6.6mm; Digikey SRR1260-1R5YTR-ND -> SRP7050TA-1R5MCT-ND
- Q1: Digikey (none) -> ZXMS6004DN8-13DICT-ND
- R2: Digikey (none) -> 13-RT0805FRE07390KLCT-ND
- R20: Digikey 311-158KCRTR-ND -> 311-300KCRCT-ND
- R21: Digikey 311-51.1KCRCT-ND -> 311-43.2KCRCT-ND
- R25: Digikey (none) -> 311-20.0KCRCT-ND
- R26, R4: Digikey (none) -> 311-10.0KCRCT-ND
- R3: Digikey (none) -> 311-1.00KCRCT-ND
- R5: Digikey 311-120CRCT-ND -> 13-RT0805FRE07120RLCT-ND
- R53, R54, R59: renamed from R?; footprint (none) -> Resistor_SMD:R_0805_2012Metric; Digikey (none) -> 311-10.0KCRCT-ND
- SW3: renamed from SW2; Digikey (none) -> CKN10723CT-ND
- U11: Digikey (none) -> LM2664M6/NOPBCT-ND
- U14: Digikey (none) -> 296-TPS259620DDARCT-ND
- U15: Digikey (none) -> 296-27463-1-ND
- U2: Digikey ISL3175EIBZ-TCT-ND -> 1016-1150-5-ND
- U3: Digikey (none) -> ADA4861-3YRZ-RL7CT-ND
- U3: Digikey ADA4891-3ARZ-ND -> ADA4861-3YRZ-RL7CT-ND
- U4: Digikey 1727-3464-ND -> 296-8201-1-ND
- U4: footprint (none) -> Package_SO:SOIC-14_3.9x8.7mm_P1.27mm; Digikey (none) -> 296-8201-1-ND
- gave numbers to parts that had none: 5
Connections:
- net +12V: now also U1.5 (GAIN_SEL)
- net GND: now also SW1.2 (B), SW2.2 (B); no longer U1.5 (GAIN_SEL)
- net blank: now also U4.3, U4.4
- net sense_0v: no longer U10.17 (GPIO13)
- net sense_2.5v: no longer U10.19 (GPIO14)
- net red_fb: now reaches R12.2, R15.2, U3.6 (-)
- net green_ac: now reaches C40.1, Q6.3 (D), R59.1, U3.12 (+)
- net green_fb: now reaches R13.2, R16.2, U3.13 (-)
- net blue_ac: now reaches C38.1, Q4.3 (D), R53.1, U3.10 (+)
- net blue_fb: now reaches R11.2, R14.2, U3.9 (-)
- net red_ac: now reaches C39.1, Q5.3 (D), R54.1, U3.5 (+)
- net at U10.21 (GPIO16): now also SW2.1 (A)
- net at U10.22 (GPIO17): now also SW1.1 (A)
- no-connect marks 55 -> 64

Commit message: final edits
Parts:
- added R60: 330, Resistor_SMD:R_0805_2012Metric, symbol Device:R
- C24, C25, C26, C27: value 2.2uF -> 2.2uF 50V; Digikey 1276-3362-1-ND -> 1276-2884-1-ND
- R11, R12, R13: Digikey 311-100CRCT-ND -> 311-330CRCT-ND
- R52: Digikey 311-10.0KCRCT-ND -> 311-100CRCT-ND
Connections:
- net sense_0v: now also U10.17 (GPIO13)
- net at Q1.7 (D1), Q1.8 (D1), R52.1: now also R60.2; no longer J2.1 (VBUS)
- new net: J2.1 (VBUS), R60.1
- no-connect marks 64 -> 63
Changed lines of the file:
@@
 F 2 "Resistor_SMD:R_0805_2012Metric" V 8130 11950 50  0001 C CNN
 F 3 "~" H 8200 11950 50  0001 C CNN
-F 4 "311-100CRCT-ND" H 8200 11950 50  0001 C CNN "Digikey"
+F 4 "311-330CRCT-ND" H 8200 11950 50  0001 C CNN "Digikey"
 	1    8200 11950
 	-1   0    0    1
@@
 F 2 "Resistor_SMD:R_0805_2012Metric" V 8130 13500 50  0001 C CNN
 F 3 "~" H 8200 13500 50  0001 C CNN
-F 4 "311-100CRCT-ND" H 8200 13500 50  0001 C CNN "Digikey"
+F 4 "311-330CRCT-ND" H 8200 13500 50  0001 C CNN "Digikey"
 	1    8200 13500
 	-1   0    0    1
@@
 F 2 "Resistor_SMD:R_0805_2012Metric" V 8080 15050 50  0001 C CNN
 F 3 "~" H 8150 15050 50  0001 C CNN
-F 4 "311-100CRCT-ND" H 8150 15050 50  0001 C CNN "Digikey"
+F 4 "311-330CRCT-ND" H 8150 15050 50  0001 C CNN "Digikey"
 	1    8150 15050
 	-1   0    0    1
@@
 	10000 6100 10500 6100
 Wire Wire Line
-	10500 6100 10500 6950
-Wire Wire Line
 	11500 6950 10500 6950
-Connection ~ 10500 6950
 Text Label 10200 7150 2    50   ~ 0
 sense_0v
@@
 F 2 "Resistor_SMD:R_0805_2012Metric" V 11430 7200 50  0001 C CNN
 F 3 "~" H 11500 7200 50  0001 C CNN
-F 4 "311-10.0KCRCT-ND" H 11500 7200 50  0001 C CNN "Digikey"
+F 4 "311-100CRCT-ND" H 11500 7200 50  0001 C CNN "Digikey"
 	1    11500 7200
 	1    0    0    -1
@@
 P 5900 4400
 F 0 "C24" H 6015 4446 50  0000 L CNN
-F 1 "2.2uF" H 6015 4355 50  0000 L CNN
+F 1 "2.2uF 50V" H 6015 4355 50  0000 L CNN
 F 2 "Capacitor_SMD:C_1210_3225Metric" H 5938 4250 50  0001 C CNN
 F 3 "~" H 5900 4400 50  0001 C CNN
-F 4 "1276-3362-1-ND" H 5900 4400 50  0001 C CNN "Digikey"
+F 4 "1276-2884-1-ND" H 5900 4400 50  0001 C CNN "Digikey"
 	1    5900 4400
 	1    0    0    -1
@@
 P 6200 4400
 F 0 "C25" H 6315 4446 50  0000 L CNN
-F 1 "2.2uF" H 6315 4355 50  0000 L CNN
+F 1 "2.2uF 50V" H 6315 4355 50  0000 L CNN
 F 2 "Capacitor_SMD:C_1210_3225Metric" H 6238 4250 50  0001 C CNN
 F 3 "~" H 6200 4400 50  0001 C CNN
-F 4 "1276-3362-1-ND" H 6200 4400 50  0001 C CNN "Digikey"
+F 4 "1276-2884-1-ND" H 6200 4400 50  0001 C CNN "Digikey"
 	1    6200 4400
 	1    0    0    -1
@@
 P 6500 4400
 F 0 "C26" H 6615 4446 50  0000 L CNN
-F 1 "2.2uF" H 6615 4355 50  0000 L CNN
+F 1 "2.2uF 50V" H 6615 4355 50  0000 L CNN
 F 2 "Capacitor_SMD:C_1210_3225Metric" H 6538 4250 50  0001 C CNN
 F 3 "~" H 6500 4400 50  0001 C CNN
-F 4 "1276-3362-1-ND" H 6500 4400 50  0001 C CNN "Digikey"
+F 4 "1276-2884-1-ND" H 6500 4400 50  0001 C CNN "Digikey"
 	1    6500 4400
 	1    0    0    -1
@@
 P 6800 4400
 F 0 "C27" H 6915 4446 50  0000 L CNN
-F 1 "2.2uF" H 6915 4355 50  0000 L CNN
+F 1 "2.2uF 50V" H 6915 4355 50  0000 L CNN
 F 2 "Capacitor_SMD:C_1210_3225Metric" H 6838 4250 50  0001 C CNN
 F 3 "~" H 6800 4400 50  0001 C CNN
-F 4 "1276-3362-1-ND" H 6800 4400 50  0001 C CNN "Digikey"
+F 4 "1276-2884-1-ND" H 6800 4400 50  0001 C CNN "Digikey"
 	1    6800 4400
 	1    0    0    -1
@@
 	1    0    0    -1
 $EndComp
-NoConn ~ 13800 8700
 NoConn ~ 13800 8900
 $Comp
@@
 Wire Wire Line
 	12450 8500 12450 8600
+Text Label 13800 8700 2    50   ~ 0
+sense_0v
+$Comp
+L Device:R R60
+U 1 1 607A2180
+P 10500 6800
+F 0 "R60" H 10570 6846 50  0000 L CNN
+F 1 "330" H 10570 6755 50  0000 L CNN
+F 2 "Resistor_SMD:R_0805_2012Metric" V 10430 6800 50  0001 C CNN
+F 3 "~" H 10500 6800 50  0001 C CNN
+F 4 "311-330CRCT-ND" H 10500 6800 50  0001 C CNN "Digikey"
+	1    10500 6800
+	1    0    0    -1
+$EndComp
+Connection ~ 10500 6950
+Wire Wire Line
+	10500 6100 10500 6650
 $EndSCHEMATC

Commit message: add todos
Other:
- note added: "TODO:\nreverse amp PLIMIT\nleave video amp disables floating\nremove R60"
Changed lines of the file:
@@
 Wire Wire Line
 	10500 6100 10500 6650
+Text Notes 4050 8000 0    50   ~ 0
+TODO:\nreverse amp PLIMIT\nleave video amp disables floating\nremove R60
 $EndSCHEMATC

Commit message: BOM changes
Parts:
- C12, C9: Digikey 1276-1782-1-ND -> 1276-1092-1-ND
- J1: Digikey WM14667-ND -> SAM10870-ND
- J2: Digikey ED2982-ND -> SAM10873-ND
- L2, L3, L4, L5: Digikey 811-3582-2-ND -> 811-3582-1-ND
- R32: value 91k -> 1k; Digikey 311-91.0KCRCT-ND -> 311-1.00KCRCT-ND
- R33: value 20k -> 220; Digikey 311-20.0KCRCT-ND -> 311-220CRCT-ND
- R60: value 330 -> 0; Digikey 311-330CRCT-ND -> 311-0.0ARCT-ND‎
Changed lines of the file:
@@
 F 2 "Connector_USB:USB_B_OST_USB-B1HSxx_Horizontal" H 9850 6250 50  0001 C CNN
 F 3 " ~" H 9850 6250 50  0001 C CNN
-F 4 "ED2982-ND" H 9700 6300 50  0001 C CNN "Digikey"
+F 4 "SAM10873-ND" H 9700 6300 50  0001 C CNN "Digikey"
 	1    9700 6300
 	1    0    0    -1
@@
 F 2 "Capacitor_SMD:C_1210_3225Metric" H 21638 1450 50  0001 C CNN
 F 3 "~" H 21600 1600 50  0001 C CNN
-F 4 "1276-1782-1-ND " H 21600 1600 50  0001 C CNN "Digikey"
+F 4 "1276-1092-1-ND" H 21600 1600 50  0001 C CNN "Digikey"
 	1    21600 1600
 	1    0    0    -1
@@
 P 22050 1600
 F 0 "R32" H 22120 1646 50  0000 L CNN
-F 1 "91k" H 22120 1555 50  0000 L CNN
+F 1 "1k" H 22120 1555 50  0000 L CNN
 F 2 "Resistor_SMD:R_0805_2012Metric" V 21980 1600 50  0001 C CNN
 F 3 "~" H 22050 1600 50  0001 C CNN
-F 4 "311-91.0KCRCT-ND" H 22050 1600 50  0001 C CNN "Digikey"
+F 4 "311-1.00KCRCT-ND" H 22050 1600 50  0001 C CNN "Digikey"
 	1    22050 1600
 	1    0    0    -1
@@
 P 22050 2150
 F 0 "R33" H 22120 2196 50  0000 L CNN
-F 1 "20k" H 22120 2105 50  0000 L CNN
+F 1 "220" H 22120 2105 50  0000 L CNN
 F 2 "Resistor_SMD:R_0805_2012Metric" V 21980 2150 50  0001 C CNN
 F 3 "~" H 22050 2150 50  0001 C CNN
-F 4 "311-20.0KCRCT-ND" H 22050 2150 50  0001 C CNN "Digikey"
+F 4 "311-220CRCT-ND" H 22050 2150 50  0001 C CNN "Digikey"
 	1    22050 2150
 	1    0    0    -1
@@
 F 2 "Capacitor_SMD:C_1210_3225Metric" H 17688 1450 50  0001 C CNN
 F 3 "~" H 17650 1600 50  0001 C CNN
-F 4 "1276-1782-1-ND " H 17650 1600 50  0001 C CNN "Digikey"
+F 4 "1276-1092-1-ND" H 17650 1600 50  0001 C CNN "Digikey"
 	1    17650 1600
 	1    0    0    -1
@@
 F 2 "Connector_USB:USB_A_Molex_67643_Horizontal" H 9850 5100 50  0001 C CNN
 F 3 " ~" H 9850 5100 50  0001 C CNN
-F 4 "WM14667-ND" H 9700 5150 50  0001 C CNN "Digikey"
+F 4 "SAM10870-ND" H 9700 5150 50  0001 C CNN "Digikey"
 	1    9700 5150
 	1    0    0    -1
@@
 F 2 "Inductor_SMD:L_7.3x7.3_H4.5" H 5650 3750 50  0001 C CNN
 F 3 "~" H 5650 3750 50  0001 C CNN
-F 4 "811-3582-2-ND" V 5650 3750 50  0001 C CNN "Digikey"
+F 4 "811-3582-1-ND" V 5650 3750 50  0001 C CNN "Digikey"
 	1    5650 3750
 	0    -1   -1   0
@@
 F 2 "Inductor_SMD:L_7.3x7.3_H4.5" H 5650 3850 50  0001 C CNN
 F 3 "~" H 5650 3850 50  0001 C CNN
-F 4 "811-3582-2-ND" H 5650 3850 50  0001 C CNN "Digikey"
+F 4 "811-3582-1-ND" H 5650 3850 50  0001 C CNN "Digikey"
 	1    5650 3850
 	0    -1   -1   0
@@
 F 2 "Inductor_SMD:L_7.3x7.3_H4.5" H 5650 4050 50  0001 C CNN
 F 3 "~" H 5650 4050 50  0001 C CNN
-F 4 "811-3582-2-ND" H 5650 4050 50  0001 C CNN "Digikey"
+F 4 "811-3582-1-ND" H 5650 4050 50  0001 C CNN "Digikey"
 	1    5650 4050
 	0    -1   -1   0
@@
 F 2 "Inductor_SMD:L_7.3x7.3_H4.5" H 5650 4150 50  0001 C CNN
 F 3 "~" H 5650 4150 50  0001 C CNN
-F 4 "811-3582-2-ND" H 5650 4150 50  0001 C CNN "Digikey"
+F 4 "811-3582-1-ND" H 5650 4150 50  0001 C CNN "Digikey"
 	1    5650 4150
 	0    -1   -1   0
@@
 P 10500 6800
 F 0 "R60" H 10570 6846 50  0000 L CNN
-F 1 "330" H 10570 6755 50  0000 L CNN
+F 1 "0" H 10570 6755 50  0000 L CNN
 F 2 "Resistor_SMD:R_0805_2012Metric" V 10430 6800 50  0001 C CNN
 F 3 "~" H 10500 6800 50  0001 C CNN
-F 4 "311-330CRCT-ND" H 10500 6800 50  0001 C CNN "Digikey"
+F 4 "311-0.0ARCT-ND‎" H 10500 6800 50  0001 C CNN "Digikey"
 	1    10500 6800
 	1    0    0    -1
