File: td-io.kicad_pcb (KiCad board)
At the start: 2 copper layers, 200 x 75 mm, 121 parts, among them J1 USB_A, J2 USB_B, J3 JAMMA_Edge, J4 Conn_Coaxial, J5 DB15_Female_HighDensity, J6 Conn_02x04_Top_Bottom, J7 Conn_02x17_Odd_Even, J8 Conn_Coaxial, J9 Conn_01x04_Male, Q1 FDS6930B, Q2 ZXMS6004DN8, Q3 ZXMS6004DN8, SW1 SW_DIP_x02, SW2 SW_DIP_x01, U1 TPA3138D2, U10 Pico, U11 TL081, U12 CPC1017N, U13 74LS165, U2 SP3481CN, U3 ADA4891-3, U4 74LS86, U5 AT24CS01-SSHM, U6 74LS165, U7 TPS568230, U8 74LS165, U9 74LS165

Commit message: changes
Parts:
- removed J8: Conn_Coaxial, td-io:CUI_RCJ-01X
- removed R53: 20k, Resistor_SMD:R_0805_2012Metric
- removed R54: 10k, Resistor_SMD:R_0805_2012Metric
- added C28: 3.3uF, Capacitor_SMD:C_0805_2012Metric, F.Cu at (197.8, 106.5)
- added C29: 0.1uF, Capacitor_SMD:C_0805_2012Metric, F.Cu at (95.0, 121.3)
- added C30: 3.3uF, Capacitor_SMD:C_0805_2012Metric, F.Cu at (194.8, 103.8)
- added C31: 3.3uF, Capacitor_SMD:C_0805_2012Metric, F.Cu at (191.6, 106.2)
- added C32: 0.1uF, Capacitor_SMD:C_0805_2012Metric, F.Cu at (262.3, 98.7)
- added R2: 400k, Resistor_SMD:R_0805_2012Metric, F.Cu at (105.9, 135.7)
- added R3: 1k, Resistor_SMD:R_0805_2012Metric, F.Cu at (105.9, 138.0)
- added R4: 10k, Resistor_SMD:R_0805_2012Metric, F.Cu at (207.5, 110.5)
- added U14: TPS259620, Package_SO:SOIC-8-1EP_3.9x4.9mm_P1.27mm_EP2.41x3.3mm_ThermalVias, F.Cu at (100.3, 138.7)
- added U15: LM2903, Package_SO:SOIC-8_3.9x4.9mm_P1.27mm, F.Cu at (214.2, 110.7)
- C12, C9: footprint Capacitor_SMD:C_1206_3216Metric -> Capacitor_SMD:C_1210_3225Metric
- C17, C18: value 100uF -> 100uF 16V
- C24, C25, C26, C27: footprint Capacitor_SMD:C_0805_2012Metric -> Capacitor_SMD:C_1210_3225Metric
- J4: value Conn_Coaxial -> Conn_Coaxial_x2; footprint td-io:CUI_RCJ-01X -> td-io:PJRAN2X1U01AUX
- J5: value DB15_Female_HighDensity -> DB15_Female_HighDensity_MountingHoles
- J9: footprint Connector_JST:JST_EH_B4B-EH-A_1x04_P2.50mm_Vertical -> td-io:JST_SH_B4B-NH-A_1x04_P2.50mm_Vertical
- L1: value 1uH -> 1.5uH; footprint Inductor_SMD:L_7.3x7.3_H3.5 -> Inductor_SMD:L_Bourns_SRR1260
- R11, R12, R13: value 100 -> 330
- R17, R18, R19: value R -> 75
- R20: value 160k -> 300k
- R21: value 51k -> 43k
- R25: value 1k -> 20k
- R26: value 1k -> 10k
- R32: value 90k -> 91k
- R52: value 10k -> 100
- R55: value R -> 1k
- U1: footprint Package_SO:HTSSOP-28-1EP_4.4x9.7mm_P0.65mm_EP2.85x5.4mm_ThermalVias -> td-io:HTSSOP-28-1EP_4.4x9.7mm_P0.65mm_tpa3138_ThermalVias
- U11: value TL081 -> LM2664M4; footprint Package_SO:SOIC-8_3.9x4.9mm_P1.27mm -> Package_TO_SOT_SMD:SOT-23-6
- U2: value SP3481CN -> ISL3175EIBZ-T
- U3: value ADA4891-3 -> ADA4861-3
- U7: footprint Package_DFN_QFN:VQFN-20-1EP_3x3mm_P0.45mm_EP1.55x1.55mm_ThermalVias -> td-io:RJE-20
- moved R26 87.8 mm to (207.5, 117.9), turned to 270 degrees
- moved R25 87.4 mm to (207.5, 114.2), turned to 270 degrees
- moved C3 46.7 mm to (216.2, 106.5), turned to 180 degrees
- moved RV1 44.6 mm to (116.8, 132.0), turned to 180 degrees
- moved R33 22.6 mm to (102.0, 122.0), turned to 0 degrees
- moved U11 20.7 mm to (194.6, 107.0), turned to 0 degrees
- moved C9 20.5 mm to (94.5, 124.0), turned to 0 degrees
- moved J4 20.2 mm to (158.5, 86.0), turned to 180 degrees
- moved R32 19.0 mm to (101.9, 119.0), turned to 180 degrees
- moved SW2 18.4 mm to (135.0, 93.0), turned to 270 degrees
- moved R20 16.0 mm to (101.9, 116.1), turned to 0 degrees
- moved C23 15.8 mm to (142.5, 103.3)
- moved C2 15.6 mm to (128.9, 98.0), turned to 180 degrees
- moved C8 15.5 mm to (129.1, 94.7), turned to 180 degrees
- moved R21 15.1 mm to (103.2, 113.5), turned to 180 degrees
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Connections:
- C19 pad 1: /speaker+ -> Net-(C19-Pad1)
- C20 pad 1: /speaker_r- -> Net-(C20-Pad1)
- C22 pad 1: /speaker- -> Net-(C22-Pad1)
- C23 pad 1: /speaker_r+ -> Net-(C23-Pad1)
- C3 pad 1: +3V3 -> +5V
- C6 pad 2: GND -> -5V
- C9 pad 1: +5V -> +5VL
- J3 pad 3: +5V -> +5VL
- J3 pad 4: +5V -> +5VL
- J3 pad C: +5V -> +5VL
- J3 pad D: +5V -> +5VL
- J4 pad 1: Net-(C2-Pad2) -> /r_in
- J4 pad 2: GND -> /l_in
- J5 pad 0: (no net) -> GND
- J5 pad 11: /vga_vsync -> Net-(J5-Pad11)
- J5 pad 14: Net-(J5-Pad14) -> /vga_vsync
- J6 pad 3: +5V -> +5VL
- L2 pad 1: Net-(L2-Pad1) -> Net-(C19-Pad1)
- L3 pad 1: Net-(L3-Pad1) -> Net-(C22-Pad1)
- L4 pad 1: Net-(L4-Pad1) -> Net-(C20-Pad1)
- L5 pad 1: Net-(L5-Pad1) -> Net-(C23-Pad1)
- Q1 pad 3: Net-(D1-Pad1) -> Net-(Q1-Pad3)
- Q1 pad 4: /sense_2.5v -> Net-(Q1-Pad4)
- Q1 pad 5: Net-(J2-Pad1) -> Net-(Q1-Pad5)
- Q1 pad 6: Net-(J2-Pad1) -> Net-(Q1-Pad5)
- R25 pad 2: Net-(C2-Pad1) -> Net-(R25-Pad2)
- R26 pad 1: Net-(R26-Pad1) -> Net-(R25-Pad2)
- R26 pad 2: Net-(C8-Pad1) -> GND
- R52 pad 1: /sense_2.5v -> Net-(J2-Pad1)
- R52 pad 2: GND -> Net-(D1-Pad1)
- R55 pad 1: Net-(J1-Pad3) -> +3V3
- RV1 pad 1: Net-(R25-Pad1) -> GND
- RV1 pad 2: Net-(RV1-Pad2) -> Net-(C2-Pad2)
- RV1 pad 3: GND -> /l_in
- RV1 pad 4: Net-(R26-Pad1) -> GND
- RV1 pad 5: Net-(RV1-Pad5) -> Net-(C8-Pad2)
- RV1 pad 6: GND -> /r_in
- SW2 pad 1: Net-(RV1-Pad5) -> Net-(C8-Pad1)
- SW2 pad 2: Net-(RV1-Pad2) -> Net-(C2-Pad1)
- U1 pad 12: Net-(RV1-Pad5) -> Net-(C8-Pad1)
- U1 pad 18: Net-(L5-Pad1) -> Net-(C23-Pad1)
- U1 pad 20: Net-(L4-Pad1) -> Net-(C20-Pad1)
- U1 pad 23: Net-(L3-Pad1) -> Net-(C22-Pad1)
- U1 pad 25: Net-(L2-Pad1) -> Net-(C19-Pad1)
- U1 pad 3: Net-(RV1-Pad2) -> Net-(C2-Pad1)
- U10 pad 1: /jvs_rx -> /jvs_tx
- U10 pad 15: Net-(U10-Pad15) -> /sense_in_high
- U10 pad 16: Net-(U10-Pad16) -> /sense_in_low
- U10 pad 2: /jvs_tx -> /jvs_rx
- U10 pad 24: Net-(U10-Pad24) -> /sr_clk
- U10 pad 26: Net-(U10-Pad26) -> /sr_data
- U10 pad 27: Net-(U10-Pad27) -> /sr_clr
- U10 pad 31: /sense_in -> Net-(U10-Pad31)
- U10 pad 6: /sr_clr -> Net-(U10-Pad6)
- U10 pad 7: /sr_clk -> Net-(U10-Pad7)
- U10 pad 9: /sr_data -> Net-(U10-Pad9)
- U11 pad 1: Net-(U11-Pad1) -> GND
- U11 pad 2: Net-(R53-Pad1) -> -5V
- U11 pad 3: GND -> Net-(C30-Pad2)
- U11 pad 4: GND -> +5V
- U11 pad 5: Net-(U11-Pad5) -> +5V
- U11 pad 6: /sense_in -> Net-(C30-Pad1)
- U2 pad 6: Net-(J1-Pad2) -> Net-(J1-Pad3)
- U2 pad 7: Net-(J1-Pad3) -> Net-(J1-Pad2)
- U3 pad 1: GND -> +5V
- U3 pad 11: GND -> -5V
- U3 pad 2: GND -> +5V
- U3 pad 3: GND -> +5V
- U4 pad 10: (no net) -> GND
- U4 pad 11: (no net) -> Net-(U4-Pad11)
- U4 pad 12: (no net) -> GND
- U4 pad 13: (no net) -> GND
- U4 pad 14: (no net) -> +5V
- U4 pad 7: (no net) -> GND
- U4 pad 8: (no net) -> Net-(U4-Pad8)
- U4 pad 9: (no net) -> GND
- U7 pad 12: +5V -> +5VL
- U7 pad 2: +5V -> +5VL
- U7 pad 3: +5V -> +5VL
- U7 pad 4: +5V -> +5VL
- U7 pad 5: +5V -> +5VL
Routing:
- net +5VL: track 0.00 -> 116.2 mm, vias 0 -> 2
- net +5V: track 414.4 -> 311.1 mm, vias 10 -> 9
- net /r_in: track 0.00 -> 80.8 mm
- net /l_in: track 0.00 -> 64.0 mm
- net +3V3: track 286.2 -> 347.4 mm, vias 38 -> 36
- net /sense_in: track 51.4 -> 0.00 mm, vias 2 -> 0
- net Net-(RV1-Pad2): track 41.6 -> 0.00 mm, vias 2 -> 0
- net Net-(RV1-Pad5): track 40.9 -> 0.00 mm, vias 2 -> 0
- net /sr_clk: track 144.9 -> 112.7 mm
- net Net-(C8-Pad2): track 60.9 -> 29.7 mm
- net /sense_2.5v: track 30.9 -> 0.00 mm
- net /sr_data: track 58.6 -> 32.4 mm
- net Net-(C8-Pad1): track 2.60 -> 27.0 mm
- net Net-(C2-Pad1): track 2.60 -> 26.5 mm
- net /sr_clr: track 146.9 -> 124.3 mm
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- added copper zone on F.Cu, net +5VL
- added copper zone on F.Cu, net /speaker+
- removed copper zone on F.Cu, net +3.3VP
- removed copper zone on B.Cu, net +5V
- removed copper zone on F.Cu, net +5V
- removed copper zone on F.Cu, net /SW
- removed copper zone on F.Cu, net Net-(L2-Pad1)
- removed copper zone on F.Cu, net Net-(L3-Pad1)
- removed copper zone on F.Cu, net Net-(L4-Pad1)
- removed copper zone on F.Cu, net Net-(L5-Pad1)

Commit message: change switch
Parts:
- added C33: 3.3uF, Capacitor_SMD:C_0805_2012Metric, F.Cu at (175.5, 113.0)
- added C34: 0.1uF, Capacitor_SMD:C_0805_2012Metric, F.Cu at (159.0, 97.5)
- added C35: 0.1uF, Capacitor_SMD:C_0805_2012Metric, F.Cu at (144.4, 97.5)
- added C36: 47uF 16V, Capacitor_SMD:C_1210_3225Metric, F.Cu at (137.8, 97.5)
- added C37: 47uF 16V, Capacitor_SMD:C_1210_3225Metric, F.Cu at (165.6, 97.5)
- C17, C18: value 100uF 16V -> 47uF 16V; footprint Capacitor_SMD:C_1206_3216Metric -> Capacitor_SMD:C_1210_3225Metric
- SW2: value SW_DIP_x01 -> SW_DPDT_x2; footprint Button_Switch_SMD:SW_DIP_SPSTx01_Slide_Omron_A6S-110x_W8.9mm_P2.54mm -> Button_Switch_SMD:SW_DPDT_CK_JS202011JCQN
- moved C21 4.66 mm to (136.2, 90.7), turned to 270 degrees
- moved C1 3.36 mm to (165.8, 94.0), turned to 180 degrees
- moved C17 3.18 mm to (162.0, 97.5)
- moved R1 3.12 mm to (162.1, 94.0)
- moved C10 3.00 mm to (103.2, 113.5)
- moved C11 3.00 mm to (89.9, 119.5)
- moved C29 3.00 mm to (95.0, 124.3)
- moved C9 3.00 mm to (94.5, 127.0)
- moved L1 3.00 mm to (94.5, 110.4)
- moved R20 3.00 mm to (101.9, 119.1)
- moved R21 3.00 mm to (103.2, 116.5)
- moved R32 3.00 mm to (101.9, 122.0)
- moved R33 3.00 mm to (102.0, 125.0)
- moved SW2 3.00 mm to (132.0, 93.0), turned to 90 degrees
- moved U7 3.00 mm to (97.2, 121.0)
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Connections:
- SW2 pad 1: Net-(C8-Pad1) -> Net-(C2-Pad1)
- SW2 pad 2: Net-(C2-Pad1) -> Net-(C8-Pad1)
Routing:
- net +5VL: track 116.2 -> 162.1 mm, vias 2 -> 13
- net +3.3VP: track 33.4 -> 56.7 mm, vias 0 -> 4
- net +12V: track 203.5 -> 218.2 mm, vias 5 -> 6
- net Net-(C2-Pad1): track 26.5 -> 31.4 mm
- net GND: track 111.9 -> 107.1 mm, vias 55 -> 53
- net Net-(R1-Pad1): track 4.38 -> 7.19 mm
- net Net-(C21-Pad2): track 13.8 -> 16.6 mm
- net Net-(C1-Pad2): track 10.9 -> 13.5 mm
- net +5V: track 311.1 -> 312.9 mm
- net Net-(C8-Pad1): track 27.0 -> 25.5 mm
- net Net-(C8-Pad2): track 29.7 -> 29.0 mm
- net Net-(C2-Pad2): track 28.0 -> 27.4 mm
- added copper zone on F.Cu, net /SW
- removed copper zone on F.Cu, net /speaker+
Other:
- board text added: "+3.3V 8A +5V 10A +12V 2A"
- board text added: "JVS ONLY"
- board text added: "speaker output"
- board text added: "td-io v1.1 2021 https://github.com/tdaede/td-io CERN-OHL-W"
- board text added: "volume"
- board text removed: "td-io v1.0 2021 https://github.com/tdaede/td-io CERN-OHL-W"

Commit message: Move some tracks around
Parts:
- added J8: Conn_01x05_Male, Connector_PinHeader_2.54mm:PinHeader_1x05_P2.54mm_Vertical, F.Cu at (247.1, 101.5)
- moved R52 17.1 mm to (230.4, 99.2), turned to 0 degrees
Connections:
- U10 pad 31: Net-(U10-Pad31) -> /adc0
- U10 pad 32: Net-(U10-Pad32) -> /adc1
- U10 pad 34: Net-(U10-Pad34) -> /adc2
Routing:
- net /adc2: track 0.00 -> 25.4 mm
- net /adc1: track 0.00 -> 25.4 mm
- net /adc0: track 0.00 -> 25.4 mm
- net +3V3: track 347.4 -> 359.9 mm
- net Net-(D1-Pad1): track 13.4 -> 2.99 mm
- net Net-(J2-Pad1): track 19.6 -> 24.7 mm
Other:
- board text added: "adc"

Commit message: more fixes
Parts:
- added C38: 1uF, Capacitor_SMD:C_0805_2012Metric, F.Cu at (183.0, 104.0)
- added C39: 1uF, Capacitor_SMD:C_0805_2012Metric, F.Cu at (191.0, 104.0)
- added C40: 1uF, Capacitor_SMD:C_0805_2012Metric, F.Cu at (175.0, 104.0)
- added Q4: 2N7002NXBKR, Package_TO_SOT_SMD:SOT-23, F.Cu at (187.0, 103.0)
- added Q5: 2N7002NXBKR, Package_TO_SOT_SMD:SOT-23, F.Cu at (195.0, 103.0)
- added Q6: 2N7002NXBKR, Package_TO_SOT_SMD:SOT-23, F.Cu at (179.0, 103.0)
- added R53: 10k, Resistor_SMD:R_0805_2012Metric, F.Cu at (183.0, 107.5)
- added R54: 10k, Resistor_SMD:R_0805_2012Metric, F.Cu at (191.0, 107.5)
- added R59: 10k, Resistor_SMD:R_0805_2012Metric, F.Cu at (175.0, 107.5)
- added SW2: SW_DPDT_x2, Button_Switch_SMD:SW_DPDT_CK_JS202011JCQN, F.Cu at (215.5, 126.5)
- L1: footprint Inductor_SMD:L_Bourns_SRR1260 -> Inductor_SMD:L_Bourns_SRP7028A_7.3x6.6mm
- Q1: value FDS6930B -> ZXMS6004DN8
- SW1: value SW_DIP_x02 -> SW_DPDT_x2; footprint Button_Switch_SMD:SW_DIP_SPSTx02_Slide_Omron_A6S-210x_W8.9mm_P2.54mm -> Button_Switch_SMD:SW_DPDT_CK_JS202011JCQN
- moved C30 12.0 mm to (188.2, 113.8), turned to 270 degrees
- moved C31 11.1 mm to (191.2, 117.2), turned to 180 degrees
- moved R12 8.80 mm to (195.1, 107.5)
- moved C28 8.08 mm to (190.9, 110.8), turned to 180 degrees
- moved U11 7.70 mm to (191.4, 114.0), turned to 90 degrees
- moved R18 7.44 mm to (181.2, 119.1), turned to 90 degrees
- moved R11 5.60 mm to (187.0, 107.5)
- moved C12 5.43 mm to (97.4, 106.4)
- moved SW1 5.32 mm to (210.0, 126.5), turned to 90 degrees
- moved R19 4.96 mm to (176.8, 119.1), turned to 90 degrees
- moved U5 4.68 mm to (210.0, 103.7)
- moved R10 4.66 mm to (175.0, 100.5)
- moved R17 4.65 mm to (185.6, 119.1), turned to 90 degrees
- moved R14 4.40 mm to (187.8, 119.1), turned to 270 degrees
- moved R13 4.34 mm to (179.0, 107.5)
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- renumbered SW2 to SW3
Connections:
- net /sense_2.5v renamed Net-(U10-Pad19)
- net Net-(R11-Pad2) renamed /blue_fb
- net Net-(R12-Pad2) renamed /red_fb
- net Net-(R13-Pad2) renamed /green_fb
- net Net-(U4-Pad3) renamed /blank
- SW1 pad 1: GND -> Net-(SW1-Pad1)
- SW1 pad 4: Net-(SW1-Pad4) -> (no net)
- U1 pad 5: GND -> +12V
- U10 pad 17: /sense_0v -> Net-(U10-Pad17)
- U10 pad 21: Net-(SW1-Pad4) -> Net-(SW2-Pad1)
- U10 pad 22: Net-(SW1-Pad3) -> Net-(SW1-Pad1)
- U3 pad 10: /vga_blue -> /blue_ac
- U3 pad 12: /vga_green -> /green_ac
- U3 pad 5: /vga_red -> /red_ac
Routing:
- net /blank: track 1.27 -> 33.1 mm, vias 0 -> 4
- net /red_ac: track 0.00 -> 19.9 mm
- net +5V: track 312.9 -> 293.5 mm
- net Net-(SW1-Pad1): track 0.00 -> 18.5 mm
- net /green_ac: track 0.00 -> 18.0 mm
- net Net-(R14-Pad1): track 29.1 -> 14.7 mm, vias 0 -> 2
- net Net-(SW1-Pad3): track 14.4 -> 0.00 mm
- net /blue_ac: track 0.00 -> 12.4 mm
- net /vga_red: track 19.9 -> 8.35 mm, vias 1 -> 0
- net Net-(J1-Pad1): track 45.0 -> 34.3 mm, vias 1 -> 3
- net /jamma_red: track 88.2 -> 78.5 mm, vias 2 -> 0
- net Net-(U10-Pad9): track 9.57 -> 0.00 mm, vias 2 -> 0
- net Net-(SW2-Pad1): track 0.00 -> 8.86 mm
- net /sense_0v: track 17.1 -> 9.47 mm
- net Net-(SW1-Pad4): track 7.25 -> 0.00 mm
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Other:
- board text added: "1"
- board text added: "2"
- board text added: "coin chutes"
- board text added: "on"

Commit message: final edits
Parts:
- added R60: 330, Resistor_SMD:R_0805_2012Metric, F.Cu at (240.2, 92.4)
Connections:
- Q1 pad 7: Net-(J2-Pad1) -> Net-(Q1-Pad7)
- Q1 pad 8: Net-(J2-Pad1) -> Net-(Q1-Pad7)
- R52 pad 1: Net-(J2-Pad1) -> Net-(Q1-Pad7)
- U10 pad 17: Net-(U10-Pad17) -> /sense_0v
Routing:
- net Net-(Q1-Pad7): track 0.00 -> 14.8 mm
- net Net-(J2-Pad1): track 24.7 -> 11.5 mm
- net +5VL: track 157.4 -> 166.9 mm
- net /sense_0v: track 9.47 -> 16.8 mm
- net Net-(J1-Pad2): track 53.9 -> 54.8 mm

Commit message: changes for 1.2
Parts:
- removed R60: 330, Resistor_SMD:R_0805_2012Metric
- added JP1: Jumper_NC_Small, Jumper:SolderJumper-2_P1.3mm_Bridged_RoundedPad1.0x1.5mm, F.Cu at (265.5, 133.5)
- added R61: 10k, Resistor_SMD:R_0805_2012Metric, F.Cu at (214.9, 91.8)
- added R62: 10k, Resistor_SMD:R_0805_2012Metric, F.Cu at (215.0, 95.0)
- added R63: 200k, Resistor_SMD:R_0805_2012Metric, F.Cu at (205.5, 102.0)
- added U16: PCA9306D, Package_SO:SO-8_3.9x4.9mm_P1.27mm, F.Cu at (201.5, 104.0)
- C24, C25, C26, C27: value 2.2uF -> 2.2uF 50V
- D2: value BAT54A -> BAT54C
- R32: value 91k -> 1k
- R33: value 20k -> 220
- U11: value LM2664M4 -> MAX1720EUT
- moved C7 4.21 mm to (205.5, 106.2)
- moved D2 1.00 mm to (269.0, 134.0), turned to 0 degrees
- moved J9 0.50 mm to (147.5, 121.0)
Connections:
- net Net-(C7-Pad1) renamed +5VD
- net Net-(J5-Pad12) renamed /vga_sda
- net Net-(J5-Pad15) renamed /vga_scl
- D2 pad 2: Net-(D2-Pad2) -> +5V
- D2 pad 3: +5V -> Net-(D2-Pad3)
- Q1 pad 7: Net-(Q1-Pad7) -> Net-(J2-Pad1)
- Q1 pad 8: Net-(Q1-Pad7) -> Net-(J2-Pad1)
- R52 pad 1: Net-(Q1-Pad7) -> Net-(J2-Pad1)
- U1 pad 10: GND -> +12V
- U10 pad 39: Net-(D2-Pad2) -> Net-(D2-Pad3)
- U10 pad 6: Net-(U10-Pad6) -> /i2c_sda
- U10 pad 7: Net-(U10-Pad7) -> /i2c_scl
- U11 pad 1: GND -> -5V
- U11 pad 2: -5V -> +5V
- U11 pad 4: +5V -> GND
- U3 pad 1: +5V -> Net-(U3-Pad1)
- U3 pad 2: +5V -> Net-(U3-Pad2)
- U3 pad 3: +5V -> Net-(U3-Pad3)
Routing:
- net +5VD: track 16.0 -> 115.8 mm, vias 1 -> 4
- net /i2c_sda: track 0.00 -> 77.9 mm, vias 0 -> 4
- net /i2c_scl: track 0.00 -> 75.1 mm, vias 0 -> 4
- net +3V3: track 362.4 -> 395.5 mm
- net Net-(Q1-Pad7): track 14.8 -> 0.00 mm
- net Net-(J2-Pad1): track 11.5 -> 24.7 mm
- net /vga_scl: track 14.2 -> 27.3 mm, vias 0 -> 2
- net /vga_sda: track 23.5 -> 35.6 mm, vias 0 -> 2
- net Net-(D2-Pad3): track 0.00 -> 9.16 mm
- net Net-(D2-Pad2): track 9.16 -> 0.00 mm
- net Net-(R63-Pad2): track 0.00 -> 7.89 mm
- net +12V: track 219.6 -> 223.5 mm, vias 7 -> 8
- net GND: track 106.2 -> 103.7 mm, vias 97 -> 96
- net Net-(D2-Pad1): track 0.00 -> 1.97 mm
- net /meter2_ctl: track 124.4 -> 123.0 mm
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Other:
- board text added: "td-io v1.2 2021 https://github.com/tdaede/td-io CERN-OHL-W"
- board text removed: "td-io v1.1 2021 https://github.com/tdaede/td-io CERN-OHL-W"
