File: td-io.kicad_sch (KiCad schematic)
At the start: 141 parts, among them J1 USB_A, J2 USB_B, J3 JAMMA_Edge, J4 Conn_Coaxial_x2, J5 DB15_Female_HighDensity_Mount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, J6 Conn_02x04_Top_Bottom, J7 Conn_02x17_Odd_Even, J8 DNP, J9 Conn_01x04_Male, Q1 AO4818B, Q2 AO4818B, Q3 AO4818B, Q4 2N7002NXBKR, Q5 2N7002NXBKR, Q6 2N7002NXBKR, SW1 SW_DPDT_x2, SW2 SW_DPDT_x2, SW3 SW_DPDT_x2, U1 TPA3138D2, U10 Pico, U11 MAX860, U12 CPC1017N, U13 74LV165, U15 LM2903, U16 PCA9306D, U2 ISL3175EIBZ-T, U3 ADA4861-3, U4 74LS86, U6 74LV165, U8 74LV165, U9 74LV165

Commit message: forking it hard
Parts:
- removed C1, C19, C2, C20, C21, C22, C23, C38, C39, C4, C40, C8: 1uF, Capacitor_SMD:C_0805_2012Metric, symbol Device:C
- removed C13, C14, C15, C16, C3, C32, C34, C35, C5, C6, C7: 0.1uF, Capacitor_SMD:C_0805_2012Metric, symbol Device:C
- removed C17, C18, C36, C37: 47uF 16V, Capacitor_SMD:C_1210_3225Metric, symbol Device:C
- removed C24, C25, C26, C27: 2.2uF 50V, Capacitor_SMD:C_1210_3225Metric, symbol Device:C
- removed C28, C30, C31, C33: 3.3uF, Capacitor_SMD:C_0805_2012Metric, symbol Device:C
- removed D2: BAT54C, Package_TO_SOT_SMD:SOT-23, symbol Diode:BAT54C
- removed D3, D4: MMBZ18VALT1G, Package_TO_SOT_SMD:SOT-23, symbol Power_Protection:SP0502BAHT
- removed F2, F3, F4, F5, F6: Polyfuse, Resistor_SMD:R_1812_4532Metric, symbol Device:Polyfuse
- removed H1, H2, H3, H4: MountingHole_Pad, MountingHole:MountingHole_3.2mm_M3_Pad_Via, symbol Mechanical:MountingHole_Pad
- removed J1: USB_A, Connector_USB:USB_A_Molex_67643_Horizontal, symbol Connector:USB_A
- removed J3: JAMMA_Edge, td-io:JAMMA, symbol td-io:JAMMA_Edge
- removed J4: Conn_Coaxial_x2, td-io:PJRAN2X1U01AUX, symbol Connector:Conn_Coaxial_x2
- removed J5: DB15_Female_HighDensity_MountingHoles, td-io:DSUB-15-HD_Female_Horizontal_P2.29x2.5mm_EdgePinOffset8.35mm_Housed_MountingHolesOffset10.89mm, symbol Connector:DB15_Female_HighDensity_MountingHoles
- removed J6: Conn_02x04_Top_Bottom, td-io:B08P-VL, symbol Connector_Generic:Conn_02x04_Top_Bottom
- removed J7: Conn_02x17_Odd_Even, td-io:DF1BZ-34DP-2.5DS, symbol Connector_Generic:Conn_02x17_Odd_Even
- removed J8: DNP, Connector_PinHeader_2.54mm:PinHeader_1x05_P2.54mm_Vertical, symbol Connector:Conn_01x05_Male
- removed J9: Conn_01x04_Male, td-io:JST_SH_B4B-NH-A_1x04_P2.50mm_Vertical, symbol Connector:Conn_01x04_Male
- removed L2, L3, L4, L5: 15uH, Inductor_SMD:L_7.3x7.3_H4.5, symbol Device:L
- removed Q2, Q3: AO4818B, Package_SO:SOIC-8_3.9x4.9mm_P1.27mm, symbol Transistor_FET:FDS6930B
- removed Q4, Q5, Q6: 2N7002NXBKR, Package_TO_SOT_SMD:SOT-23, symbol Transistor_FET:2N7002
- removed R1, R22, R23, R24, R26, R27, R28, R29, R30, R31, R34, R35, R36, R37, R38, R39, R4, R40, R41, R42, R43, R44, R45, R46, R47, R48, R49, R51, R53, R54, R56, R57, R58, R59, R6, R61, R62, R7: 10k, Resistor_SMD:R_0805_2012Metric, symbol Device:R
- removed R10, R17, R18, R19, R8, R9: 75, Resistor_SMD:R_0805_2012Metric, symbol Device:R
- removed R11, R12, R13: 330, Resistor_SMD:R_0805_2012Metric, symbol Device:R
- removed R14, R15, R16: 1k, Resistor_SMD:R_0805_2012Metric, symbol Device:R
- removed R25: 20k, Resistor_SMD:R_0805_2012Metric, symbol Device:R
- removed R63: 200k, Resistor_SMD:R_0805_2012Metric, symbol Device:R
- removed RV1: R_POT_Dual, td-io:PTV112-4420A-A503, symbol Device:R_Potentiometer_Dual
- removed SW1, SW2, SW3: SW_DPDT_x2, Button_Switch_SMD:SW_DPDT_CK_JS202011JCQN, symbol Switch:SW_DPDT_x2
- removed U1: TPA3138D2, td-io:HTSSOP-28-1EP_4.4x9.7mm_P0.65mm_tpa3138_ThermalVias, symbol td-io:TPA3138D2
- removed U10: Pico, RPi_Pico:RPi_Pico_SMD_TH, symbol MCU_RaspberryPi_and_Boards:Pico
- removed U11: MAX860, Package_SO:SOIC-8_3.9x4.9mm_P1.27mm, symbol Converter_DCDC:TC7662Bx0A
- removed U13, U6, U8, U9: 74LV165, Package_SO:SOIC-16_3.9x9.9mm_P1.27mm, symbol 74xx:74LS165
- removed U15: LM2903, Package_SO:SOIC-8_3.9x4.9mm_P1.27mm, symbol Comparator:LM2903
- removed U16: PCA9306D, Package_SO:SO-8_3.9x4.9mm_P1.27mm, symbol Interface:PCA9306D
- removed U3: ADA4861-3, Package_SO:SOIC-14_3.9x8.7mm_P1.27mm, symbol td-io:ADA4891-3
- removed U4: 74LS86, Package_SO:SOIC-14_3.9x8.7mm_P1.27mm, symbol 74xx:74LS86
- added J1: Conn_01x04, Connector_PinHeader_2.54mm:PinHeader_1x04_P2.54mm_Vertical, symbol Connector_Generic:Conn_01x04
- added J3, J4: Conn_01x02, Connector_PinHeader_2.54mm:PinHeader_1x02_P2.54mm_Vertical, symbol Connector_Generic:Conn_01x02
- Q1: ShittyBackup (none) -> NTMD6N02R2G
- U12: Backup (none) -> CPC1002NTR; Backup2 (none) -> CLA153-ND
Connections:
- net +3V3: now also J3.1 (Pin_1)
- net GND: now also J3.2 (Pin_2)
- net jvs_de: now also J1.3 (Pin_3)
- net jvs_re: now also J1.2 (Pin_2)
- net jvs_rx: now also J1.1 (Pin_1)
- net jvs_tx: now also J1.4 (Pin_4)
- net sense_0v: now also J4.2 (Pin_2)
- net termination: now also J4.1 (Pin_1)
- no-connect marks 61 -> 5
Other:
- removed sheet JVS Power
- moved on the sheet: Q1B

Commit message: Update td-io.kicad_sch
Parts:
- removed F1: Polyfuse, Resistor_SMD:R_1812_4532Metric, symbol Device:Polyfuse
Connections:
- net at J2.1 (VBUS): now also Q1.7 (D1), Q1.8 (D1), R52.1
Changed lines of the file:
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@@
     (title "TD-IO")
   )
+  (junction (at 266.7 189.23) (diameter 0) (color 0 0 0 0)
+  )
+  (junction (at 293.37 134.62) (diameter 0) (color 0 0 0 0)
+  )
   (junction (at 266.7 176.53) (diameter 0) (color 0 0 0 0)
-  )
-  (junction (at 266.7 189.23) (diameter 0) (color 0 0 0 0)
-  )
-  (junction (at 293.37 134.62) (diameter 0) (color 0 0 0 0)
   )
   (junction (at 295.91 162.56) (diameter 0) (color 0 0 0 0)
@@
     (stroke (width 0) (type default) (color 0 0 0 0))
   )
-  (wire (pts (xy 266.7 154.94) (xy 266.7 168.91))
+  (wire (pts (xy 266.7 154.94) (xy 266.7 176.53))
     (stroke (width 0) (type default) (color 0 0 0 0))
   )
@@
     (pin "2")
   )
-  (symbol (lib_id "Device:Polyfuse") (at 266.7 172.72 0) (unit 1)
-    (in_bom yes) (on_board yes) (fields_autoplaced)
-    (property "Reference" "F1" (id 0) (at 268.859 171.8853 0)
-      (effects (font (size 1.27 1.27)) (justify left))
-    )
-    (property "Value" "Polyfuse" (id 1) (at 268.859 174.4222 0)
-      (effects (font (size 1.27 1.27)) (justify left))
-    )
-    (property "Footprint" "Resistor_SMD:R_1812_4532Metric" (id 2) (at 267.97 177.8 0)
-      (effects (font (size 1.27 1.27)) (justify left) hide)
-    )
-    (property "Datasheet" "~" (id 3) (at 266.7 172.72 0)
-      (effects (font (size 1.27 1.27)) hide)
-    )
-    (property "Digikey" "507-1762-1-ND" (id 4) (at 266.7 172.72 0)
-      (effects (font (size 1.27 1.27)) hide)
-    )
-    (pin "1")
-    (pin "2")
-  )
   (symbol (lib_id "power:+3.3V") (at 310.515 183.515 0) (unit 1)
     (in_bom yes) (on_board yes)
@@
       (reference "D1") (unit 2) (value "BAV99S") (footprint "Package_TO_SOT_SMD:SOT-363_SC-70-6")
     )
-    (path "/a0c827a5-01f0-47ad-a296-ca35a9634660"
-      (reference "F1") (unit 1) (value "Polyfuse") (footprint "Resistor_SMD:R_1812_4532Metric")
-    )
     (path "/189480db-1242-4a6d-9914-c371e53a85b9"
