File: td-io.kicad_sch (KiCad schematic)
At the start: 141 parts, among them J1 USB_A, J2 USB_B, J3 JAMMA_Edge, J4 Conn_Coaxial_x2, J5 DB15_Female_HighDensity_Mount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, J6 Conn_02x04_Top_Bottom, J7 Conn_02x17_Odd_Even, J8 DNP, J9 Conn_01x04_Male, Q1 AO4818B, Q2 AO4818B, Q3 AO4818B, Q4 2N7002NXBKR, Q5 2N7002NXBKR, Q6 2N7002NXBKR, SW1 SW_DPDT_x2, SW2 SW_DPDT_x2, SW3 SW_DPDT_x2, U1 TPA3138D2, U10 Pico, U11 MAX860, U12 CPC1017N, U13 74LV165, U15 LM2903, U16 PCA9306D, U2 ISL3175EIBZ-T, U3 ADA4861-3, U4 74LS86, U6 74LV165, U8 74LV165, U9 74LV165

Commit message: Update PCB to v1.4
Parts:
- U10: footprint RPi_Pico:RPi_Pico_SMD_TH -> td-io:RPi_Pico_SMD
- U11: value MAX860 -> MAX860ISA+T; Digikey MAX860IUA+CT-ND -> MAX860ISA+TCT-ND
- U2: value ISL3175EIBZ-T -> ISL3178EIBZ-T; Digikey 1016-1150-5-ND -> 20-ISL3178EIBZ-TCT-ND
Connections:
- net +12V: no longer U1.1 (NC), U1.10 (PLIMIT)
- net +5V: now also U11.7 (OSC)
- net at R1.1, U1.2 (~{SD2/FAULT}): now also U1.1 (NC)
- net at C21.2, U1.9 (GVDD): now also U1.10 (PLIMIT)
- net +3V3 renamed +3.3V
Other:
- note added: "TODO: remember to connect EN to VIN on SiC437 Scoot potentiometer inwards"
